File: Cube/PCB/Cube-8x8x8-512_LEDS.sch (KiCad schematic (older format))
At the start: 3 parts

Commit message: Update
Update
Parts:
- removed J?: Conn_01x05_Male, symbol Conn_01x05_Male
- added J2: Conn_01x06_Male, symbol Conn_01x06_Male
- added R1: 1K, symbol R
- added SW1, SW2: Chevron, symbol Chevron
- gave numbers to parts that had none: 2
Connections:
- net +5V: now also J2.1 (Pin_1), SW2.1
- net GND: now also J2.6 (Pin_6)
- net Matrice/QH'_OUT: now also J2.2 (Pin_2)
- net RCLK_CMD: now also J2.4 (Pin_4)
- net SRCLK_CMD: now also J2.3 (Pin_3)
- net SER_CMD_A: now reaches XA1.D12
- net SER_CMD_A: now also J2.5 (Pin_5), SW1.1
- new net: R1.2, SW1.2, SW2.2
- new net Matrice/~SRCLR_IN: R1.1
Changed lines of the file:
@@
 LIBS:valves
 LIBS:alex-library
+LIBS:Cube-8x8x8-512_LEDS-cache
 EELAYER 25 0
 EELAYER END
@@
 $EndDescr
 $Comp
-L Conn_01x02_Male J?
+L Conn_01x02_Male J1
 U 1 1 5B220BC5
 P 1300 800
-F 0 "J?" H 1300 900 50  0000 C CNN
+F 0 "J1" H 1300 900 50  0000 C CNN
 F 1 "Conn_01x02_Male" H 1300 600 50  0000 C CNN
 F 2 "" H 1300 800 50  0001 C CNN
@@
 $EndComp
 $Comp
-L VCC #PWR?
+L VCC #PWR1
 U 1 1 5B220C09
 P 1700 750
-F 0 "#PWR?" H 1700 600 50  0001 C CNN
+F 0 "#PWR1" H 1700 600 50  0001 C CNN
 F 1 "VCC" H 1700 900 50  0000 C CNN
 F 2 "" H 1700 750 50  0001 C CNN
@@
 $EndComp
 $Comp
-L GND #PWR?
+L GND #PWR2
 U 1 1 5B220C1F
 P 1700 950
-F 0 "#PWR?" H 1700 700 50  0001 C CNN
+F 0 "#PWR2" H 1700 700 50  0001 C CNN
 F 1 "GND" H 1700 800 50  0000 C CNN
 F 2 "" H 1700 950 50  0001 C CNN
@@
 $EndSheet
 $Comp
-L VCC #PWR?
+L VCC #PWR3
 U 1 1 5B222EBC
 P 2000 750
-F 0 "#PWR?" H 2000 600 50  0001 C CNN
+F 0 "#PWR3" H 2000 600 50  0001 C CNN
 F 1 "VCC" H 2000 900 50  0000 C CNN
 F 2 "" H 2000 750 50  0001 C CNN
@@
 $EndComp
 $Comp
-L +5V #PWR?
+L +5V #PWR6
 U 1 1 5B222F9E
 P 3550 750
-F 0 "#PWR?" H 3550 600 50  0001 C CNN
+F 0 "#PWR6" H 3550 600 50  0001 C CNN
 F 1 "+5V" H 3550 890 50  0000 C CNN
 F 2 "" H 3550 750 50  0001 C CNN
@@
 Power Supply\n9-12V
 $Sheet
-S 7050 750  1500 400
+S 7050 750  1450 600
 U 5B22355E
 F0 "Matrice" 60
@@
 F3 "RCLK_IN" I L 7050 950 60
 F4 "SER_IN" I L 7050 1100 60
-F5 "QH'_OUT" O R 8550 1100 60
+F5 "QH'_OUT" O R 8500 1250 60
+F6 "~SRCLR_IN" I L 7050 1250 60
 $EndSheet
 $Comp
-L Arduino_Uno_Shield XA?
+L Arduino_Uno_Shield XA1
 U 1 1 5B270BF1
 P 4750 4350
-F 0 "XA?" V 4850 4350 60  0000 C CNN
+F 0 "XA1" V 4850 4350 60  0000 C CNN
 F 1 "Arduino_Uno_Shield" V 4650 4350 60  0000 C CNN
 F 2 "" H 6550 8100 60  0001 C CNN
@@
 $EndComp
 $Comp
-L VCC #PWR?
+L VCC #PWR5
 U 1 1 5B27111A
 P 2950 5350
-F 0 "#PWR?" H 2950 5200 50  0001 C CNN
+F 0 "#PWR5" H 2950 5200 50  0001 C CNN
 F 1 "VCC" H 2950 5500 50  0000 C CNN
 F 2 "" H 2950 5350 50  0001 C CNN
@@
 $EndComp
 $Comp
-L GND #PWR?
+L GND #PWR4
 U 1 1 5B27258E
 P 2950 4900
-F 0 "#PWR?" H 2950 4650 50  0001 C CNN
+F 0 "#PWR4" H 2950 4650 50  0001 C CNN
 F 1 "GND" H 2950 4750 50  0000 C CNN
 F 2 "" H 2950 4900 50  0001 C CNN
@@
 Text GLabel 6650 4250 2    60   Output ~ 0
 SER_CMD
-Text GLabel 6650 4400 2    60   Output ~ 0
+Text GLabel 6650 4550 2    60   Output ~ 0
 SRCLK_CMD
 Wire Wire Line
@@
 Wire Wire Line
 	6550 4250 6650 4250
-Wire Wire Line
-	6050 4400 6650 4400
 Text GLabel 6850 1100 0    60   Input ~ 0
 SER_CMD
@@
 	6850 1100 7050 1100
 $Comp
-L +5V #PWR?
+L +5V #PWR8
 U 1 1 5B273801
-P 9050 950
-F 0 "#PWR?" H 9050 800 50  0001 C CNN
-F 1 "+5V" H 9050 1090 50  0000 C CNN
-F 2 "" H 9050 950 50  0001 C CNN
-F 3 "" H 9050 950 50  0001 C CNN
-	1    9050 950
-	1    0    0    -1
-$EndComp
-$Comp
-L GND #PWR?
+P 9150 1100
+F 0 "#PWR8" H 9150 950 50  0001 C CNN
+F 1 "+5V" H 9150 1240 50  0000 C CNN
+F 2 "" H 9150 1100 50  0001 C CNN
+F 3 "" H 9150 1100 50  0001 C CNN
+	1    9150 1100
+	1    0    0    -1
+$EndComp
+$Comp
+L GND #PWR9
 U 1 1 5B273B6C
-P 9050 1550
-F 0 "#PWR?" H 9050 1300 50  0001 C CNN
-F 1 "GND" H 9050 1400 50  0000 C CNN
-F 2 "" H 9050 1550 50  0001 C CNN
-F 3 "" H 9050 1550 50  0001 C CNN
-	1    9050 1550
-	1    0    0    -1
-$EndComp
-Wire Wire Line
-	8550 1100 9250 1100
-Wire Wire Line
-	9050 950  9050 1000
-Wire Wire Line
-	9050 1000 9250 1000
-Text GLabel 8550 1450 0    60   Input ~ 0
+P 9150 2050
+F 0 "#PWR9" H 9150 1800 50  0001 C CNN
+F 1 "GND" H 9150 1900 50  0000 C CNN
+F 2 "" H 9150 2050 50  0001 C CNN
+F 3 "" H 9150 2050 50  0001 C CNN
+	1    9150 2050
+	1    0    0    -1
+$EndComp
+Wire Wire Line
+	9150 1100 9150 1150
+Wire Wire Line
+	9150 1150 9350 1150
+Text GLabel 8550 1700 0    60   Input ~ 0
 RCLK_CMD
-Text GLabel 8550 1300 0    60   Input ~ 0
+Text GLabel 8550 1550 0    60   Input ~ 0
 SRCLK_CMD
-$Comp
-L Conn_01x05_Male J?
-U 1 1 5B276725
-P 9450 1200
-F 0 "J?" H 9450 1500 50  0000 C CNN
-F 1 "Conn_01x05_Male" H 9450 900 50  0000 C CNN
-F 2 "" H 9450 1200 50  0001 C CNN
-F 3 "" H 9450 1200 50  0001 C CNN
-	1    9450 1200
+Wire Wire Line
+	8700 1350 9350 1350
+Wire Wire Line
+	8750 1450 9350 1450
+Wire Wire Line
+	8500 1250 9350 1250
+Wire Wire Line
+	8700 1350 8700 1550
+Wire Wire Line
+	8700 1550 8550 1550
+Wire Wire Line
+	8750 1450 8750 1700
+Wire Wire Line
+	8750 1700 8550 1700
+Text GLabel 5550 1600 0    60   Input ~ 0
+SER_CMD_A
+Text GLabel 6650 4400 2    60   Output ~ 0
+SER_CMD_A
+Wire Wire Line
+	6050 4300 6500 4300
+Wire Wire Line
+	6500 4300 6500 4400
+Wire Wire Line
+	6500 4400 6650 4400
+Wire Wire Line
+	6050 4400 6450 4400
+Wire Wire Line
+	6450 4400 6450 4550
+Wire Wire Line
+	6450 4550 6650 4550
+$Comp
+L Conn_01x06_Male J2
+U 1 1 5B2604EF
+P 9550 1350
+F 0 "J2" H 9550 1650 50  0000 C CNN
+F 1 "Conn_01x06_Male" H 9550 950 50  0000 C CNN
+F 2 "" H 9550 1350 50  0001 C CNN
+F 3 "" H 9550 1350 50  0001 C CNN
+	1    9550 1350
 	-1   0    0    -1
 $EndComp
 Wire Wire Line
-	8550 1300 8600 1300
-Wire Wire Line
-	8600 1300 8600 1200
-Wire Wire Line
-	8600 1200 9250 1200
-Wire Wire Line
-	8550 1450 8650 1450
-Wire Wire Line
-	8650 1450 8650 1300
-Wire Wire Line
-	8650 1300 9250 1300
-Wire Wire Line
-	9050 1550 9050 1400
-Wire Wire Line
-	9050 1400 9250 1400
+	9150 2050 9150 1650
+Wire Wire Line
+	9150 1650 9350 1650
+Text GLabel 8550 1850 0    60   Input ~ 0
+SER_CMD_A
+Wire Wire Line
+	8550 1850 8800 1850
+Wire Wire Line
+	8800 1850 8800 1550
+Wire Wire Line
+	8800 1550 9350 1550
+$Comp
+L R R1
+U 1 1 5B2396A1
+P 6400 1600
+F 0 "R1" V 6480 1600 50  0000 C CNN
+F 1 "1K" V 6400 1600 50  0000 C CNN
+F 2 "" V 6330 1600 50  0001 C CNN
+F 3 "" H 6400 1600 50  0001 C CNN
+	1    6400 1600
+	0    1    1    0
+$EndComp
+$Comp
+L Chevron SW1
+U 1 1 5B23982B
+P 5800 1600
+F 0 "SW1" H 5800 1500 60  0000 C CNN
+F 1 "Chevron" H 5800 1700 60  0000 C CNN
+F 2 "" H 5900 1600 60  0001 C CNN
+F 3 "" H 5900 1600 60  0001 C CNN
+	1    5800 1600
+	1    0    0    -1
+$EndComp
+$Comp
+L Chevron SW2
+U 1 1 5B2399AD
+P 6000 1400
+F 0 "SW2" H 6000 1300 60  0000 C CNN
+F 1 "Chevron" H 6000 1500 60  0000 C CNN
+F 2 "" H 6100 1400 60  0001 C CNN
+F 3 "" H 6100 1400 60  0001 C CNN
+	1    6000 1400
+	0    1    1    0
+$EndComp
+$Comp
+L +5V #PWR7
+U 1 1 5B239BE5
+P 6000 1200
+F 0 "#PWR7" H 6000 1050 50  0001 C CNN
+F 1 "+5V" H 6000 1340 50  0000 C CNN
+F 2 "" H 6000 1200 50  0001 C CNN
+F 3 "" H 6000 1200 50  0001 C CNN
+	1    6000 1200
+	1    0    0    -1
+$EndComp
+Wire Wire Line
+	5550 1600 5700 1600
+Wire Wire Line
+	6000 1500 6000 1600
+Wire Wire Line
+	5900 1600 6250 1600
+Connection ~ 6000 1600
+Wire Wire Line
+	6550 1600 6900 1600
+Wire Wire Line
+	6900 1600 6900 1250
+Wire Wire Line
+	6900 1250 7050 1250
+Wire Wire Line
+	6000 1200 6000 1300
 $EndSCHEMATC

Commit message: Update project
Remove a image corrupted -_-
Parts:
- added J2: Conn_01x09_Male, alex-library:Connect-9pin, symbol Conn_01x09_Male
- added J3: Conn_01x04_Male, alex-library:Connect-4pin, symbol Conn_01x04_Male
- added J4: Conn_01x10_Male, alex-library:Connect-10pin, symbol Conn_01x10_Male
- added J5: Conn_01x06_Male, alex-library:Connect-6pin, symbol Conn_01x06_Male
- J1: footprint (none) -> alex-library:Connect-2pin
- J6: renamed from J2; footprint (none) -> alex-library:Connect-6pin
- R1: footprint (none) -> alex-library:R_Axial_Long6.3mm_Dia2.5mm_Pas15.24mm_Horizontal
- SW1, SW2: footprint (none) -> alex-library:Chevron-E1
- XA1: footprint (none) -> alex-library:Arduino_Uno_Shield
Connections:
- net +5V: now also J2.1 (Pin_1), J3.1 (Pin_1)
- net GND: now also J2.9 (Pin_9), J3.4 (Pin_4), J4.10 (Pin_10), J5.6 (Pin_6)
- net RCLK_CMD: now also J6.3 (Pin_3); no longer J6.4 (Pin_4)
- net SRCLK_CMD: now also J6.4 (Pin_4); no longer J6.3 (Pin_3)
- net VCC: now also J4.1 (Pin_1), J5.1 (Pin_1)
- net at XA1.A0: now also J2.3 (Pin_3)
- net at XA1.A1: now also J2.4 (Pin_4)
- net at XA1.A2: now also J2.5 (Pin_5)
- net at XA1.A3: now also J2.6 (Pin_6)
- net at XA1.A4: now also J2.7 (Pin_7)
- net at XA1.A5: now also J2.8 (Pin_8)
- net at XA1.AREF: now also J2.2 (Pin_2)
- net at XA1.D2 (D2_INT0): now also J4.2 (Pin_2)
- net at XA1.D3 (D3_INT1): now also J4.3 (Pin_3)
- net at XA1.D4: now also J4.4 (Pin_4)
- net at XA1.D5: now also J4.5 (Pin_5)
- net at XA1.D6: now also J4.6 (Pin_6)
- net at XA1.D7: now also J4.7 (Pin_7)
- net at XA1.D8: now also J4.8 (Pin_8)
- net at XA1.D9: now also J4.9 (Pin_9)
- net at XA1.MISO (SPI_MISO): now also J5.2 (Pin_2)
- net at XA1.MOSI (SPI_MOSI): now also J5.3 (Pin_3)
- net at XA1.RST2 (SPI_RESET): now also J5.5 (Pin_5)
- net at XA1.SCK (SPI_SCK): now also J5.4 (Pin_4)
- net at XA1.SCL: now also J3.2 (Pin_2)
- net at XA1.SDA: now also J3.3 (Pin_3)
- net SER_CMD renamed SER_START
- net SER_CMD_A renamed SRCLR_CMD
- net SRCLR_CMD: no longer J6.5 (Pin_5)

Commit message: Update project
Update
Connections:
- net Matrice/~SRCLR_IN: now also J6.5 (Pin_5)
Changed lines of the file:
@@
 encoding utf-8
 Sheet 1 12
-Title ""
-Date ""
-Rev ""
-Comp ""
+Title "Logique de commande Cube 8x8x8 512 Leds"
+Date "2018-06-21"
+Rev "1"
+Comp "FabLab19"
 Comment1 ""
 Comment2 ""
@@
 Wire Wire Line
 	9150 1650 9350 1650
-Wire Wire Line
-	8550 1850 8800 1850
-Wire Wire Line
-	8800 1850 8800 1550
-Wire Wire Line
-	8800 1550 9350 1550
 $Comp
 L R R1
@@
 	7050 1250 6900 1250
 Wire Wire Line
-	6900 1250 6900 1600
+	6900 1250 6900 1800
+Wire Wire Line
+	6900 1800 8800 1800
+Wire Wire Line
+	8800 1800 8800 1550
+Wire Wire Line
+	8800 1550 9350 1550
+Connection ~ 6900 1600
 $EndSCHEMATC
