File: Cube/PCB/Matrice.sch (KiCad schematic (older format))
At the start: 1 part

Commit message: Update
Update
Parts:
- gave numbers to parts that had none: 1
Changed lines of the file:
@@
 LIBS:valves
 LIBS:alex-library
+LIBS:Cube-8x8x8-512_LEDS-cache
 EELAYER 25 0
 EELAYER END
@@
 F12 "R_QH" O R 2650 3700 60
 F13 "R_QH'" O R 2650 3850 60
+F14 "~SRCLR" I L 1750 3450 60
 $EndSheet
 Text GLabel 2900 3850 2    60   Output ~ 0
 SER_2
-$Sheet
-S 1750 4100 900  950
-U 5B22654D
-F0 "BlockRowAnode2" 60
-F1 "Block Row Anode 2.sch" 60
-F2 "SRCLK" I L 1750 4150 60
-F3 "RCLK" I L 1750 4300 60
-F4 "SER" I L 1750 4450 60
-F5 "R_QA" O R 2650 4150 60
-F6 "R_QB" O R 2650 4250 60
-F7 "R_QC" O R 2650 4350 60
-F8 "R_QD" O R 2650 4450 60
-F9 "R_QE" O R 2650 4550 60
-F10 "R_QF" O R 2650 4650 60
-F11 "R_QG" O R 2650 4750 60
-F12 "R_QH" O R 2650 4850 60
-F13 "R_QH'" O R 2650 5000 60
-$EndSheet
 Text GLabel 1500 4150 0    60   Input ~ 0
 SRCLK
@@
 Text GLabel 2900 5000 2    60   Output ~ 0
 SER_3
-$Sheet
-S 1750 5250 900  950
-U 5B2280E3
-F0 "BlockRowAnode3" 60
-F1 "Block Row Anode 3.sch" 60
-F2 "SRCLK" I L 1750 5300 60
-F3 "RCLK" I L 1750 5450 60
-F4 "SER" I L 1750 5600 60
-F5 "R_QA" O R 2650 5300 60
-F6 "R_QB" O R 2650 5400 60
-F7 "R_QC" O R 2650 5500 60
-F8 "R_QD" O R 2650 5600 60
-F9 "R_QE" O R 2650 5700 60
-F10 "R_QF" O R 2650 5800 60
-F11 "R_QG" O R 2650 5900 60
-F12 "R_QH" O R 2650 6000 60
-F13 "R_QH'" O R 2650 6150 60
-$EndSheet
 Text GLabel 1500 5300 0    60   Input ~ 0
 SRCLK
@@
 F12 "R_QH" O R 2650 7150 60
 F13 "R_QH'" O R 2650 7300 60
+F14 "~SRCLR" I L 1750 6900 60
 $EndSheet
 Text GLabel 1500 6450 0    60   Input ~ 0
@@
 F12 "R_QH" O R 5800 3700 60
 F13 "R_QH'" O R 5800 3850 60
+F14 "~SRCLR" I L 4900 3450 60
 $EndSheet
 Text GLabel 4650 3000 0    60   Input ~ 0
@@
 F12 "R_QH" O R 5800 4850 60
 F13 "R_QH'" O R 5800 5000 60
+F14 "~SRCLR" I L 4900 4600 60
 $EndSheet
 Text GLabel 4650 4150 0    60   Input ~ 0
@@
 F12 "R_QH" O R 5800 6000 60
 F13 "R_QH'" O R 5800 6150 60
+F14 "~SRCLR" I L 4900 5750 60
 $EndSheet
 Text GLabel 4650 5300 0    60   Input ~ 0
@@
 F12 "R_QH" O R 5800 7150 60
 F13 "R_QH'" O R 5800 7300 60
+F14 "~SRCLR" I L 4900 6900 60
 $EndSheet
 Text GLabel 4650 6450 0    60   Input ~ 0
@@
 F12 "L_QH" O R 8900 3650 60
 F13 "L_QH'" O R 8900 3800 60
+F14 "R_QH'" I L 8050 3400 60
 $EndSheet
 Text GLabel 7800 2950 0    60   Input ~ 0
@@
 A51
 $Comp
-L Matrice_8x8x8_512leds M?
+L Matrice_8x8x8_512leds M1
 U 1 1 5B33DA12
 P 4300 1150
-F 0 "M?" V 4750 3925 60  0000 C CNN
+F 0 "M1" V 4750 3925 60  0000 C CNN
 F 1 "Matrice_8x8x8_512leds" V 4800 2200 60  0000 C CNN
 F 2 "" H 4700 2150 60  0001 C CNN
@@
 Text Label 3300 3700 0    60   ~ 0
 A8
+Text Label 3300 4150 0    60   ~ 0
+A9
+Text Label 3300 4250 0    60   ~ 0
+A10
+Text Label 3300 4350 0    60   ~ 0
+A11
+Text Label 3300 4450 0    60   ~ 0
+A12
+Text Label 3300 4550 0    60   ~ 0
+A13
+Text Label 3300 4650 0    60   ~ 0
+A14
+Text Label 3300 4750 0    60   ~ 0
+A15
+Text Label 3300 4850 0    60   ~ 0
+A16
+Text Label 3300 5300 0    60   ~ 0
+A17
+Text Label 3300 5400 0    60   ~ 0
+A18
+Text Label 3300 5500 0    60   ~ 0
+A19
+Text Label 3300 5600 0    60   ~ 0
+A20
+Text Label 3300 5700 0    60   ~ 0
+A21
+Text Label 3300 5800 0    60   ~ 0
+A22
+Text Label 3300 5900 0    60   ~ 0
+A23
+Text Label 3300 6000 0    60   ~ 0
+A24
+Text Label 3300 6450 0    60   ~ 0
+A25
+Text Label 3300 6550 0    60   ~ 0
+A26
+Text Label 3300 6650 0    60   ~ 0
+A27
+Text Label 3300 6750 0    60   ~ 0
+A28
+Text Label 3300 6850 0    60   ~ 0
+A29
+Text Label 3300 6950 0    60   ~ 0
+A30
+Text Label 3300 7050 0    60   ~ 0
+A31
+Text Label 3300 7150 0    60   ~ 0
+A32
+Text Label 6300 3000 0    60   ~ 0
+A33
+Text Label 6300 3100 0    60   ~ 0
+A34
+Text Label 6300 3200 0    60   ~ 0
+A35
+Text Label 6300 3300 0    60   ~ 0
+A36
+Text Label 6300 3400 0    60   ~ 0
+A37
+Text Label 6300 3500 0    60   ~ 0
+A38
+Text Label 6300 3600 0    60   ~ 0
+A39
+Text Label 6300 3700 0    60   ~ 0
+A40
+Text Label 6300 4150 0    60   ~ 0
+A41
+Text Label 6300 4250 0    60   ~ 0
+A42
+Text Label 6300 4350 0    60   ~ 0
+A43
+Text Label 6300 4450 0    60   ~ 0
+A44
+Text Label 6300 4550 0    60   ~ 0
+A45
+Text Label 6300 4650 0    60   ~ 0
+A46
+Text Label 6300 4750 0    60   ~ 0
+A47
+Text Label 6300 4850 0    60   ~ 0
+A48
+Text Label 6300 5300 0    60   ~ 0
+A49
+Text Label 6300 5400 0    60   ~ 0
+A50
+Text Label 6300 5500 0    60   ~ 0
+A51
+Text Label 6300 5600 0    60   ~ 0
+A52
+Text Label 6300 5700 0    60   ~ 0
+A53
+Text Label 6300 5800 0    60   ~ 0
+A54
+Text Label 6300 5900 0    60   ~ 0
+A55
+Text Label 6300 6000 0    60   ~ 0
+A56
+Text Label 6300 6450 0    60   ~ 0
+A57
+Text Label 6300 6550 0    60   ~ 0
+A58
+Text Label 6300 6650 0    60   ~ 0
+A59
+Text Label 6300 6750 0    60   ~ 0
+A60
+Text Label 6300 6850 0    60   ~ 0
+A61
+Text Label 6300 6950 0    60   ~ 0
+A62
+Text Label 6300 7050 0    60   ~ 0
+A63
+Text Label 6300 7150 0    60   ~ 0
+A64
+$Sheet
+S 1750 5250 900  950
+U 5B2280E3
+F0 "BlockRowAnode3" 60
+F1 "Block Row Anode 3.sch" 60
+F2 "SRCLK" I L 1750 5300 60
+F3 "RCLK" I L 1750 5450 60
+F4 "SER" I L 1750 5600 60
+F5 "R_QA" O R 2650 5300 60
+F6 "R_QB" O R 2650 5400 60
+F7 "R_QC" O R 2650 5500 60
+F8 "R_QD" O R 2650 5600 60
+F9 "R_QE" O R 2650 5700 60
+F10 "R_QF" O R 2650 5800 60
+F11 "R_QG" O R 2650 5900 60
+F12 "R_QH" O R 2650 6000 60
+F13 "R_QH'" O R 2650 6150 60
+F14 "~SRCLR" I L 1750 5750 60
+$EndSheet
+$Sheet
+S 1750 4100 900  950
+U 5B22654D
+F0 "BlockRowAnode2" 60
+F1 "Block Row Anode 2.sch" 60
+F2 "SRCLK" I L 1750 4150 60
+F3 "RCLK" I L 1750 4300 60
+F4 "SER" I L 1750 4450 60
+F5 "R_QA" O R 2650 4150 60
+F6 "R_QB" O R 2650 4250 60
+F7 "R_QC" O R 2650 4350 60
+F8 "R_QD" O R 2650 4450 60
+F9 "R_QE" O R 2650 4550 60
+F10 "R_QF" O R 2650 4650 60
+F11 "R_QG" O R 2650 4750 60
+F12 "R_QH" O R 2650 4850 60
+F13 "R_QH'" O R 2650 5000 60
+F14 "~SRCLR" I L 1750 4600 60
+$EndSheet
+Text HLabel 1500 3450 0    60   Input ~ 0
+~SRCLR_IN
+Wire Wire Line
+	1500 3450 1750 3450
+Wire Wire Line
+	1600 3450 1600 3650
+Wire Wire Line
+	1600 3650 1450 3650
+Connection ~ 1600 3450
+Text GLabel 1450 3650 0    60   Output ~ 0
+~SRCLR_CMD
+Text GLabel 1500 4600 0    60   Input ~ 0
+~SRCLR_CMD
+Wire Wire Line
+	1500 4600 1750 4600
+Text GLabel 1500 5750 0    60   Input ~ 0
+~SRCLR_CMD
+Wire Wire Line
+	1500 5750 1750 5750
+Text GLabel 1500 6900 0    60   Input ~ 0
+~SRCLR_CMD
+Wire Wire Line
+	1500 6900 1750 6900
+Text GLabel 4650 6900 0    60   Input ~ 0
+~SRCLR_CMD
+Wire Wire Line
+	4650 6900 4900 6900
+Text GLabel 4650 5750 0    60   Input ~ 0
+~SRCLR_CMD
+Wire Wire Line
+	4650 5750 4900 5750
+Text GLabel 4650 4600 0    60   Input ~ 0
+~SRCLR_CMD
+Wire Wire Line
+	4650 4600 4900 4600
+Text GLabel 4650 3450 0    60   Input ~ 0
+~SRCLR_CMD
+Wire Wire Line
+	4650 3450 4900 3450
+Text GLabel 7800 3400 0    60   Input ~ 0
+~SRCLR_CMD
+Wire Wire Line
+	7800 3400 8050 3400
 $EndSCHEMATC

Commit message: Update project
Remove a image corrupted -_-
Parts:
- added SW10, SW11, SW12, SW13, SW14, SW15, SW16, SW17, SW18, SW19, SW20, SW21, SW22, SW23, SW24, SW25, SW26, SW27, SW28, SW29, SW3, SW30, SW31, SW32, SW33, SW34, SW35, SW36, SW37, SW38, SW39, SW4, SW5, SW6, SW7, SW8, SW9: Chevron, alex-library:Chevron-E1, symbol Chevron
- M1: footprint (none) -> alex-library:Matrice-led-8x8x8_512-Leds
Connections:
- net QH'_OUT: now also SW39.2
- net RCLK: now also SW12.1, SW16.1, SW20.1, SW24.1, SW28.1, SW32.1, SW36.1, SW4.2, SW8.1
- net RCLK_IN: now also SW4.1
- net SER_2: now also SW9.1
- net SER_3: now also SW13.1
- net SER_4: now also SW17.1
- net SER_5: now also SW21.1
- net SER_6: now also SW25.1
- net SER_7: now also SW29.1
- net SER_8: now also SW33.1
- net SER_9: now also SW37.1
- net SER_IN: now also SW5.1
- net SRCLK: now also SW11.1, SW15.1, SW19.1, SW23.1, SW27.1, SW3.2, SW31.1, SW35.1, SW7.1
- net SRCLK_IN: now also SW3.1
- new net BlockLayersCatodes/RCLK: SW36.2
- new net BlockLayersCatodes/R_QH': SW39.1
- new net BlockLayersCatodes/SER: SW37.2
- new net BlockLayersCatodes/SRCLK: SW35.2
- new net BlockLayersCatodes/~SRCLR: SW38.2
- new net BlockRowAnode1/SER: SW5.2
- new net BlockRowAnode2/RCLK: SW8.2
- new net BlockRowAnode2/SER: SW9.2
- new net BlockRowAnode2/SRCLK: SW7.2
- new net BlockRowAnode2/~SRCLR: SW10.2
- new net BlockRowAnode3/RCLK: SW12.2
- new net BlockRowAnode3/SER: SW13.2
- new net BlockRowAnode3/SRCLK: SW11.2
- new net BlockRowAnode3/~SRCLR: SW14.2
- new net BlockRowAnode4/RCLK: SW16.2
- new net BlockRowAnode4/SER: SW17.2
- new net BlockRowAnode4/SRCLK: SW15.2
- new net BlockRowAnode4/~SRCLR: SW18.2
- new net BlockRowAnode5/RCLK: SW20.2
- new net BlockRowAnode5/SER: SW21.2
- new net BlockRowAnode5/SRCLK: SW19.2
- new net BlockRowAnode5/~SRCLR: SW22.2
- new net BlockRowAnode6/RCLK: SW24.2
- new net BlockRowAnode6/SER: SW25.2
- new net BlockRowAnode6/SRCLK: SW23.2
- new net BlockRowAnode6/~SRCLR: SW26.2
- new net BlockRowAnode7/RCLK: SW28.2
- new net BlockRowAnode7/SER: SW29.2
- new net BlockRowAnode7/SRCLK: SW27.2
- new net BlockRowAnode7/~SRCLR: SW30.2
- new net BlockRowAnode8/RCLK: SW32.2
- new net BlockRowAnode8/SER: SW33.2
- new net BlockRowAnode8/SRCLK: SW31.2
- new net BlockRowAnode8/~SRCLR: SW34.2
- new net ~SRCLR: SW10.1, SW14.1, SW18.1, SW22.1, SW26.1, SW30.1, SW34.1, SW38.1, SW6.2
- new net ~SRCLR_IN: SW6.1

Commit message: Update project
Update
Parts:
- removed M1: Matrice_8x8x8_512leds, alex-library:Matrice-led-8x8x8_512-Leds, symbol Matrice_8x8x8_512leds
- added J10, J11, J12, J7, J8, J9: Conn_01x10_Male, alex-library:Connect-10pin, symbol Conn_01x10_Male
- added J13: Conn_01x04_Male, alex-library:Connect-4pin, symbol Conn_01x04_Male
- added J14: Conn_01x08_Male, alex-library:Connect-8pin, symbol Conn_01x08_Male
Connections:
- net A1: now also J7.1 (Pin_1)
- net A10: now also J7.10 (Pin_10)
- net A11: now also J8.1 (Pin_1)
- net A12: now also J8.2 (Pin_2)
- net A13: now also J8.3 (Pin_3)
- net A14: now also J8.4 (Pin_4)
- net A15: now also J8.5 (Pin_5)
- net A16: now also J8.6 (Pin_6)
- net A17: now also J8.7 (Pin_7)
- net A18: now also J8.8 (Pin_8)
- net A19: now also J8.9 (Pin_9)
- net A2: now also J7.2 (Pin_2)
- net A20: now also J8.10 (Pin_10)
- net A21: now also J9.1 (Pin_1)
- net A22: now also J9.2 (Pin_2)
- net A23: now also J9.3 (Pin_3)
- net A24: now also J9.4 (Pin_4)
- net A25: now also J9.5 (Pin_5)
- net A26: now also J9.6 (Pin_6)
- net A27: now also J9.7 (Pin_7)
- net A28: now also J9.8 (Pin_8)
- net A29: now also J9.9 (Pin_9)
- net A3: now also J7.3 (Pin_3)
- net A30: now also J9.10 (Pin_10)
- net A31: now also J10.1 (Pin_1)
- net A32: now also J10.2 (Pin_2)
- net A33: now also J10.3 (Pin_3)
- net A34: now also J10.4 (Pin_4)
- net A35: now also J10.5 (Pin_5)
- net A36: now also J10.6 (Pin_6)
- net A37: now also J10.7 (Pin_7)
- net A38: now also J10.8 (Pin_8)
- net A39: now also J10.9 (Pin_9)
- net A4: now also J7.4 (Pin_4)
- net A40: now also J10.10 (Pin_10)
- net A41: now also J11.1 (Pin_1)
- net A42: now also J11.2 (Pin_2)
- net A43: now also J11.3 (Pin_3)
- net A44: now also J11.4 (Pin_4)
- net A45: now also J11.5 (Pin_5)
- net A46: now also J11.6 (Pin_6)
- net A47: now also J11.7 (Pin_7)
- net A48: now also J11.8 (Pin_8)
- net A49: now also J11.9 (Pin_9)
- net A5: now also J7.5 (Pin_5)
- net A50: now also J11.10 (Pin_10)
- net A51: now also J12.1 (Pin_1)
- net A52: now also J12.2 (Pin_2)
- net A53: now also J12.3 (Pin_3)
- net A54: now also J12.4 (Pin_4)
- net A55: now also J12.5 (Pin_5)
- net A56: now also J12.6 (Pin_6)
- net A57: now also J12.7 (Pin_7)
- net A58: now also J12.8 (Pin_8)
- net A59: now also J12.9 (Pin_9)
- net A6: now also J7.6 (Pin_6)
- net A60: now also J12.10 (Pin_10)
- net A61: now also J13.1 (Pin_1)
- net A62: now also J13.2 (Pin_2)
- net A63: now also J13.3 (Pin_3)
- net A64: now also J13.4 (Pin_4)
- net A7: now also J7.7 (Pin_7)
- net A8: now also J7.8 (Pin_8)
- net A9: now also J7.9 (Pin_9)
- net K1: now also J14.1 (Pin_1)
- net K2: now also J14.2 (Pin_2)
- net K3: now also J14.3 (Pin_3)
- net K4: now also J14.4 (Pin_4)
- net K5: now also J14.5 (Pin_5)
- net K6: now also J14.6 (Pin_6)
- net K7: now also J14.7 (Pin_7)
- net K8: now also J14.8 (Pin_8)
Changed lines of the file:
@@
 encoding utf-8
 Sheet 3 12
-Title ""
-Date ""
-Rev ""
-Comp ""
+Title "Logique de commande Cube 8x8x8 512 Leds"
+Date "2018-06-21"
+Rev "1"
+Comp "FabLab19"
 Comment1 ""
 Comment2 ""
@@
 Text Label 5800 1900 1    60   ~ 0
 A51
-$Comp
-L Matrice_8x8x8_512leds M1
-U 1 1 5B33DA12
-P 4300 1150
-F 0 "M1" V 4750 3925 60  0000 C CNN
-F 1 "Matrice_8x8x8_512leds" V 4800 2200 60  0000 C CNN
-F 2 "alex-library:Matrice-led-8x8x8_512-Leds" H 4700 2150 60  0001 C CNN
-F 3 "" H 4700 2150 60  0001 C CNN
-	1    4300 1150
-	0    -1   -1   0
-$EndComp
 Text Label 5900 1900 1    60   ~ 0
 A52
@@
 	1500 2700 1750 2700
 Connection ~ 1500 3450
+$Comp
+L Conn_01x08_Male J14
+U 1 1 5B2BEF24
+P 7200 1150
+F 0 "J14" H 7200 1550 50  0000 C CNN
+F 1 "Conn_01x08_Male" H 7200 650 50  0000 C CNN
+F 2 "alex-library:Connect-8pin" H 7200 1150 50  0001 C CNN
+F 3 "" H 7200 1150 50  0001 C CNN
+	1    7200 1150
+	1    0    0    1
+$EndComp
+$Comp
+L Conn_01x10_Male J7
+U 1 1 5B2B61E9
+P 1200 1550
+F 0 "J7" H 1100 1550 50  0000 C CNN
+F 1 "Conn_01x10_Male" H 800 1650 50  0000 C CNN
+F 2 "alex-library:Connect-10pin" H 1200 1550 50  0001 C CNN
+F 3 "" H 1200 1550 50  0001 C CNN
+	1    1200 1550
+	0    -1   1    0
+$EndComp
+$Comp
+L Conn_01x10_Male J8
+U 1 1 5B2BBC77
+P 2200 1550
+F 0 "J8" H 2150 1550 50  0000 C CNN
+F 1 "Conn_01x10_Male" H 1850 1650 50  0000 C CNN
+F 2 "alex-library:Connect-10pin" H 2200 1550 50  0001 C CNN
+F 3 "" H 2200 1550 50  0001 C CNN
+	1    2200 1550
+	0    -1   1    0
+$EndComp
+$Comp
+L Conn_01x10_Male J9
+U 1 1 5B2BCBF6
+P 3200 1550
+F 0 "J9" H 3150 1550 50  0000 C CNN
+F 1 "Conn_01x10_Male" H 2850 1650 50  0000 C CNN
+F 2 "alex-library:Connect-10pin" H 3200 1550 50  0001 C CNN
+F 3 "" H 3200 1550 50  0001 C CNN
+	1    3200 1550
+	0    -1   1    0
+$EndComp
+$Comp
+L Conn_01x10_Male J10
+U 1 1 5B2BCF48
+P 4200 1550
+F 0 "J10" H 4100 1550 50  0000 C CNN
+F 1 "Conn_01x10_Male" H 3850 1650 50  0000 C CNN
+F 2 "alex-library:Connect-10pin" H 4200 1550 50  0001 C CNN
+F 3 "" H 4200 1550 50  0001 C CNN
+	1    4200 1550
+	0    -1   1    0
+$EndComp
+$Comp
+L Conn_01x10_Male J11
+U 1 1 5B2BE067
+P 5200 1550
+F 0 "J11" H 5100 1550 50  0000 C CNN
+F 1 "Conn_01x10_Male" H 4850 1650 50  0000 C CNN
+F 2 "alex-library:Connect-10pin" H 5200 1550 50  0001 C CNN
+F 3 "" H 5200 1550 50  0001 C CNN
+	1    5200 1550
+	0    -1   1    0
+$EndComp
+$Comp
+L Conn_01x04_Male J13
+U 1 1 5B2BE6EF
+P 6900 1550
+F 0 "J13" H 6800 1550 50  0000 C CNN
+F 1 "Conn_01x04_Male" H 6550 1650 50  0000 C CNN
+F 2 "alex-library:Connect-4pin" H 6900 1550 50  0001 C CNN
+F 3 "" H 6900 1550 50  0001 C CNN
+	1    6900 1550
+	0    -1   1    0
+$EndComp
+$Comp
+L Conn_01x10_Male J12
+U 1 1 5B2BE3BD
+P 6200 1550
+F 0 "J12" H 6100 1550 50  0000 C CNN
+F 1 "Conn_01x10_Male" H 5850 1650 50  0000 C CNN
+F 2 "alex-library:Connect-10pin" H 6200 1550 50  0001 C CNN
+F 3 "" H 6200 1550 50  0001 C CNN
+	1    6200 1550
+	0    -1   1    0
+$EndComp
 $EndSCHEMATC
