File: Cube/PCB/Alimentation.sch (KiCad schematic (older format))
At the start: 10 parts

Commit message: Update
Update
Parts:
- gave numbers to parts that had none: 10
Connections:
- net GND: now also RV1.2
Changed lines of the file:
@@
 LIBS:valves
 LIBS:alex-library
+LIBS:Cube-8x8x8-512_LEDS-cache
 EELAYER 25 0
 EELAYER END
@@
 $EndDescr
 $Comp
-L D D?
+L D D1
 U 1 1 5B220C61
 P 3100 2650
-F 0 "D?" H 3100 2750 50  0000 C CNN
+F 0 "D1" H 3100 2750 50  0000 C CNN
 F 1 "1N4007" H 3100 2550 50  0000 C CNN
 F 2 "" H 3100 2650 50  0001 C CNN
@@
 $EndComp
 $Comp
-L CP C?
+L CP C1
 U 1 1 5B220D0F
 P 3750 2900
-F 0 "C?" H 3775 3000 50  0000 L CNN
+F 0 "C1" H 3775 3000 50  0000 L CNN
 F 1 "100µF/25V" H 3775 2800 50  0000 L CNN
 F 2 "" H 3788 2750 50  0001 C CNN
@@
 $EndComp
 $Comp
-L C C?
+L C C2
 U 1 1 5B220D39
 P 4850 2900
-F 0 "C?" H 4875 3000 50  0000 L CNN
+F 0 "C2" H 4875 3000 50  0000 L CNN
 F 1 "100nF" H 4875 2800 50  0000 L CNN
 F 2 "" H 4888 2750 50  0001 C CNN
@@
 $EndComp
 $Comp
-L LM317_A U?
+L LM317_A U1
 U 1 1 5B221191
 P 5850 2650
-F 0 "U?" H 5700 2775 50  0000 C CNN
+F 0 "U1" H 5700 2775 50  0000 C CNN
 F 1 "LM317_A" H 5850 2775 50  0000 L CNN
 F 2 "" H 5850 2900 50  0001 C CIN
@@
 $EndComp
 $Comp
-L D D?
+L D D2
 U 1 1 5B2212A2
 P 6700 2900
-F 0 "D?" H 6700 3000 50  0000 C CNN
+F 0 "D2" H 6700 3000 50  0000 C CNN
 F 1 "1N4007" H 6700 2800 50  0000 C CNN
 F 2 "" H 6700 2900 50  0001 C CNN
@@
 $EndComp
 $Comp
-L C C?
+L C C3
 U 1 1 5B221619
 P 7500 2900
-F 0 "C?" H 7525 3000 50  0000 L CNN
+F 0 "C3" H 7525 3000 50  0000 L CNN
 F 1 "100nF" H 7525 2800 50  0000 L CNN
 F 2 "" H 7538 2750 50  0001 C CNN
@@
 $EndComp
 $Comp
-L R R?
+L R R2
 U 1 1 5B22167B
 P 7100 2900
-F 0 "R?" V 7180 2900 50  0000 C CNN
+F 0 "R2" V 7180 2900 50  0000 C CNN
 F 1 "240" V 7100 2900 50  0000 C CNN
 F 2 "" V 7030 2900 50  0001 C CNN
@@
 $EndComp
 $Comp
-L R R?
+L R R3
 U 1 1 5B221803
 P 7100 3500
-F 0 "R?" V 7180 3500 50  0000 C CNN
+F 0 "R3" V 7180 3500 50  0000 C CNN
 F 1 "390" V 7100 3500 50  0000 C CNN
 F 2 "" V 7030 3500 50  0001 C CNN
@@
 $EndComp
 $Comp
-L POT RV?
+L POT RV1
 U 1 1 5B221B9C
 P 7100 4150
-F 0 "RV?" V 6925 4150 50  0000 C CNN
+F 0 "RV1" V 6925 4150 50  0000 C CNN
 F 1 "470" V 7000 4150 50  0000 C CNN
 F 2 "" H 7100 4150 50  0001 C CNN
@@
 Connection ~ 6700 2650
 $Comp
-L D D?
+L D D3
 U 1 1 5B221ED0
 P 8300 2650
-F 0 "D?" H 8300 2750 50  0000 C CNN
+F 0 "D3" H 8300 2750 50  0000 C CNN
 F 1 "1N4007" H 8300 2550 50  0000 C CNN
 F 2 "" H 8300 2650 50  0001 C CNN
@@
 Connection ~ 7500 2650
 $Comp
-L GND #PWR?
+L GND #PWR10
 U 1 1 5B222026
 P 3750 3200
-F 0 "#PWR?" H 3750 2950 50  0001 C CNN
+F 0 "#PWR10" H 3750 2950 50  0001 C CNN
 F 1 "GND" H 3750 3050 50  0000 C CNN
 F 2 "" H 3750 3200 50  0001 C CNN
@@
 $EndComp
 $Comp
-L GND #PWR?
+L GND #PWR11
 U 1 1 5B222056
 P 4850 3200
-F 0 "#PWR?" H 4850 2950 50  0001 C CNN
+F 0 "#PWR11" H 4850 2950 50  0001 C CNN
 F 1 "GND" H 4850 3050 50  0000 C CNN
 F 2 "" H 4850 3200 50  0001 C CNN
@@
 $EndComp
 $Comp
-L GND #PWR?
+L GND #PWR12
 U 1 1 5B222219
 P 7100 4450
-F 0 "#PWR?" H 7100 4200 50  0001 C CNN
+F 0 "#PWR12" H 7100 4200 50  0001 C CNN
 F 1 "GND" H 7100 4300 50  0000 C CNN
 F 2 "" H 7100 4450 50  0001 C CNN
@@
 $EndComp
 $Comp
-L GND #PWR?
+L GND #PWR13
 U 1 1 5B222242
 P 7500 3200
-F 0 "#PWR?" H 7500 2950 50  0001 C CNN
+F 0 "#PWR13" H 7500 2950 50  0001 C CNN
 F 1 "GND" H 7500 3050 50  0000 C CNN
 F 2 "" H 7500 3200 50  0001 C CNN
@@
 Text Notes 5450 2200 0    60   ~ 0
 V OUT = 1.25 (1+(R2/R1))
+Wire Wire Line
+	7250 4150 7350 4150
+Wire Wire Line
+	7350 4150 7350 4350
+Wire Wire Line
+	7350 4350 7100 4350
+Connection ~ 7100 4350
 $EndSCHEMATC

Commit message: Update project
Remove a image corrupted -_-
Parts:
- C1: footprint (none) -> alex-library:CP_Radial_Dia8.0mm_Pas3.50mm
- C2, C3: footprint (none) -> alex-library:C-P_5.08-L_7.5-H_6-P_2.5
- D1, D2, D3: footprint (none) -> alex-library:D_DO-41_Pas12.70mm_Horizontal
- R2, R3: footprint (none) -> alex-library:R_Axial_Long6.3mm_Dia2.5mm_Pas15.24mm_Horizontal
- RV1: footprint (none) -> alex-library:Potentiometer_Trimmer_Bourns_3296X
- U1: footprint (none) -> alex-library:TO-220_Vertical
Changed lines of the file:
@@
 F 0 "D1" H 3100 2750 50  0000 C CNN
 F 1 "1N4007" H 3100 2550 50  0000 C CNN
-F 2 "" H 3100 2650 50  0001 C CNN
+F 2 "alex-library:D_DO-41_Pas12.70mm_Horizontal" H 3100 2650 50  0001 C CNN
 F 3 "" H 3100 2650 50  0001 C CNN
 	1    3100 2650
@@
 F 0 "C1" H 3775 3000 50  0000 L CNN
 F 1 "100µF/25V" H 3775 2800 50  0000 L CNN
-F 2 "" H 3788 2750 50  0001 C CNN
+F 2 "alex-library:CP_Radial_Dia8.0mm_Pas3.50mm" H 3788 2750 50  0001 C CNN
 F 3 "" H 3750 2900 50  0001 C CNN
 	1    3750 2900
@@
 F 0 "C2" H 4875 3000 50  0000 L CNN
 F 1 "100nF" H 4875 2800 50  0000 L CNN
-F 2 "" H 4888 2750 50  0001 C CNN
+F 2 "alex-library:C-P_5.08-L_7.5-H_6-P_2.5" H 4888 2750 50  0001 C CNN
 F 3 "" H 4850 2900 50  0001 C CNN
 	1    4850 2900
@@
 F 0 "U1" H 5700 2775 50  0000 C CNN
 F 1 "LM317_A" H 5850 2775 50  0000 L CNN
-F 2 "" H 5850 2900 50  0001 C CIN
+F 2 "alex-library:TO-220_Vertical" H 5850 2900 50  0001 C CIN
 F 3 "" H 5850 2650 50  0001 C CNN
 	1    5850 2650
@@
 F 0 "D2" H 6700 3000 50  0000 C CNN
 F 1 "1N4007" H 6700 2800 50  0000 C CNN
-F 2 "" H 6700 2900 50  0001 C CNN
+F 2 "alex-library:D_DO-41_Pas12.70mm_Horizontal" H 6700 2900 50  0001 C CNN
 F 3 "" H 6700 2900 50  0001 C CNN
 	1    6700 2900
@@
 F 0 "C3" H 7525 3000 50  0000 L CNN
 F 1 "100nF" H 7525 2800 50  0000 L CNN
-F 2 "" H 7538 2750 50  0001 C CNN
+F 2 "alex-library:C-P_5.08-L_7.5-H_6-P_2.5" H 7538 2750 50  0001 C CNN
 F 3 "" H 7500 2900 50  0001 C CNN
 	1    7500 2900
@@
 F 0 "R2" V 7180 2900 50  0000 C CNN
 F 1 "240" V 7100 2900 50  0000 C CNN
-F 2 "" V 7030 2900 50  0001 C CNN
+F 2 "alex-library:R_Axial_Long6.3mm_Dia2.5mm_Pas15.24mm_Horizontal" V 7030 2900 50  0001 C CNN
 F 3 "" H 7100 2900 50  0001 C CNN
 	1    7100 2900
@@
 F 0 "R3" V 7180 3500 50  0000 C CNN
 F 1 "390" V 7100 3500 50  0000 C CNN
-F 2 "" V 7030 3500 50  0001 C CNN
+F 2 "alex-library:R_Axial_Long6.3mm_Dia2.5mm_Pas15.24mm_Horizontal" V 7030 3500 50  0001 C CNN
 F 3 "" H 7100 3500 50  0001 C CNN
 	1    7100 3500
@@
 F 0 "RV1" V 6925 4150 50  0000 C CNN
 F 1 "470" V 7000 4150 50  0000 C CNN
-F 2 "" H 7100 4150 50  0001 C CNN
+F 2 "alex-library:Potentiometer_Trimmer_Bourns_3296X" H 7100 4150 50  0001 C CNN
 F 3 "" H 7100 4150 50  0001 C CNN
 	1    7100 4150
@@
 F 0 "D3" H 8300 2750 50  0000 C CNN
 F 1 "1N4007" H 8300 2550 50  0000 C CNN
-F 2 "" H 8300 2650 50  0001 C CNN
+F 2 "alex-library:D_DO-41_Pas12.70mm_Horizontal" H 8300 2650 50  0001 C CNN
 F 3 "" H 8300 2650 50  0001 C CNN
 	1    8300 2650
@@
 Connection ~ 7500 2650
 $Comp
-L GND #PWR10
+L GND #PWR018
 U 1 1 5B222026
 P 3750 3200
-F 0 "#PWR10" H 3750 2950 50  0001 C CNN
+F 0 "#PWR018" H 3750 2950 50  0001 C CNN
 F 1 "GND" H 3750 3050 50  0000 C CNN
 F 2 "" H 3750 3200 50  0001 C CNN
@@
 $EndComp
 $Comp
-L GND #PWR11
+L GND #PWR019
 U 1 1 5B222056
 P 4850 3200
-F 0 "#PWR11" H 4850 2950 50  0001 C CNN
+F 0 "#PWR019" H 4850 2950 50  0001 C CNN
 F 1 "GND" H 4850 3050 50  0000 C CNN
 F 2 "" H 4850 3200 50  0001 C CNN
@@
 $EndComp
 $Comp
-L GND #PWR12
+L GND #PWR020
 U 1 1 5B222219
 P 7100 4450
-F 0 "#PWR12" H 7100 4200 50  0001 C CNN
+F 0 "#PWR020" H 7100 4200 50  0001 C CNN
 F 1 "GND" H 7100 4300 50  0000 C CNN
 F 2 "" H 7100 4450 50  0001 C CNN
@@
 $EndComp
 $Comp
-L GND #PWR13
+L GND #PWR021
 U 1 1 5B222242
 P 7500 3200
-F 0 "#PWR13" H 7500 2950 50  0001 C CNN
+F 0 "#PWR021" H 7500 2950 50  0001 C CNN
 F 1 "GND" H 7500 3050 50  0000 C CNN
 F 2 "" H 7500 3200 50  0001 C CNN

Commit message: Update
Update
Add New restistor in Base Q1, Q2, Q3, Q4, Q5, Q6, Q7, Q8
New version PCB
New rename components
Parts:
- removed D2: 1N4007, alex-library:D_DO-41_Pas12.70mm_Horizontal, symbol D
- removed R2: 240, alex-library:R_Axial_Long6.3mm_Dia2.5mm_Pas15.24mm_Horizontal, symbol R
- removed R3: 390, alex-library:R_Axial_Long6.3mm_Dia2.5mm_Pas15.24mm_Horizontal, symbol R
- removed RV1: 470, alex-library:Potentiometer_Trimmer_Bourns_3296X, symbol POT
- removed U1: LM317_A, alex-library:TO-220_Vertical, symbol LM317_A
- added U1: L7805, alex-library:TO-220_Vertical, symbol L7805
- renumbered D3 to D2
Connections:
- net GND: now also U1.2 (GND)
- net at C1.1, C2.1, D1.1 (K): now also U1.1 (IN)
- net at C3.1, D2.2 (A): now also U1.3 (OUT)
Changed lines of the file:
@@
-$EndComp
-$Comp
-L LM317_A U1
-U 1 1 5B221191
-P 5850 2650
-F 0 "U1" H 5700 2775 50  0000 C CNN
-F 1 "LM317_A" H 5850 2775 50  0000 L CNN
-F 2 "alex-library:TO-220_Vertical" H 5850 2900 50  0001 C CIN
-F 3 "" H 5850 2650 50  0001 C CNN
-	1    5850 2650
-	1    0    0    -1
-$EndComp
-$Comp
-L D D2
-U 1 1 5B2212A2
-P 6700 2900
-F 0 "D2" H 6700 3000 50  0000 C CNN
-F 1 "1N4007" H 6700 2800 50  0000 C CNN
-F 2 "alex-library:D_DO-41_Pas12.70mm_Horizontal" H 6700 2900 50  0001 C CNN
-F 3 "" H 6700 2900 50  0001 C CNN
-	1    6700 2900
-	0    1    1    0
 $EndComp
 $Comp
@@
 	1    0    0    -1
 $EndComp
-$Comp
-L R R2
-U 1 1 5B22167B
-P 7100 2900
-F 0 "R2" V 7180 2900 50  0000 C CNN
-F 1 "240" V 7100 2900 50  0000 C CNN
-F 2 "alex-library:R_Axial_Long6.3mm_Dia2.5mm_Pas15.24mm_Horizontal" V 7030 2900 50  0001 C CNN
-F 3 "" H 7100 2900 50  0001 C CNN
-	1    7100 2900
-	1    0    0    -1
-$EndComp
-$Comp
-L R R3
-U 1 1 5B221803
-P 7100 3500
-F 0 "R3" V 7180 3500 50  0000 C CNN
-F 1 "390" V 7100 3500 50  0000 C CNN
-F 2 "alex-library:R_Axial_Long6.3mm_Dia2.5mm_Pas15.24mm_Horizontal" V 7030 3500 50  0001 C CNN
-F 3 "" H 7100 3500 50  0001 C CNN
-	1    7100 3500
-	1    0    0    -1
-$EndComp
-$Comp
-L POT RV1
-U 1 1 5B221B9C
-P 7100 4150
-F 0 "RV1" V 6925 4150 50  0000 C CNN
-F 1 "470" V 7000 4150 50  0000 C CNN
-F 2 "alex-library:Potentiometer_Trimmer_Bourns_3296X" H 7100 4150 50  0001 C CNN
-F 3 "" H 7100 4150 50  0001 C CNN
-	1    7100 4150
-	1    0    0    -1
-$EndComp
 Wire Wire Line
 	3250 2650 5550 2650
@@
 Wire Wire Line
 	6150 2650 8150 2650
-Wire Wire Line
-	6700 2650 6700 2750
-Wire Wire Line
-	7100 2650 7100 2750
-Connection ~ 6700 2650
 $Comp
-L D D3
+L D D2
 U 1 1 5B221ED0
 P 8300 2650
-F 0 "D3" H 8300 2750 50  0000 C CNN
+F 0 "D2" H 8300 2750 50  0000 C CNN
 F 1 "1N4007" H 8300 2550 50  0000 C CNN
 F 2 "alex-library:D_DO-41_Pas12.70mm_Horizontal" H 8300 2650 50  0001 C CNN
@@
 Wire Wire Line
 	7500 2650 7500 2750
-Connection ~ 7100 2650
 Connection ~ 7500 2650
 $Comp
@@
 L GND #PWR020
 U 1 1 5B222219
-P 7100 4450
-F 0 "#PWR020" H 7100 4200 50  0001 C CNN
-F 1 "GND" H 7100 4300 50  0000 C CNN
-F 2 "" H 7100 4450 50  0001 C CNN
-F 3 "" H 7100 4450 50  0001 C CNN
-	1    7100 4450
+P 5850 3200
+F 0 "#PWR020" H 5850 2950 50  0001 C CNN
+F 1 "GND" H 5850 3050 50  0000 C CNN
+F 2 "" H 5850 3200 50  0001 C CNN
+F 3 "" H 5850 3200 50  0001 C CNN
+	1    5850 3200
 	1    0    0    -1
 $EndComp
@@
 	4850 3050 4850 3200
 Wire Wire Line
-	5850 2950 5850 3800
-Wire Wire Line
-	5850 3800 7100 3800
-Wire Wire Line
-	7100 3650 7100 4000
-Connection ~ 7100 3800
-Wire Wire Line
-	7100 3050 7100 3350
-Wire Wire Line
-	6700 3050 6700 3800
-Connection ~ 6700 3800
-Wire Wire Line
 	7500 3050 7500 3200
-Wire Wire Line
-	7100 4300 7100 4450
 Text HLabel 2250 2650 0    60   Input ~ 0
 V_IN
@@
 Text Notes 5450 2200 0    60   ~ 0
 V OUT = 1.25 (1+(R2/R1))
+$Comp
+L L7805 U1
+U 1 1 5B743536
+P 5850 2650
+F 0 "U1" H 5700 2775 50  0000 C CNN
+F 1 "L7805" H 5850 2775 50  0000 L CNN
+F 2 "alex-library:TO-220_Vertical" H 5875 2500 50  0001 L CIN
+F 3 "" H 5850 2600 50  0001 C CNN
+	1    5850 2650
+	1    0    0    -1
+$EndComp
 Wire Wire Line
-	7250 4150 7350 4150
-Wire Wire Line
-	7350 4150 7350 4350
-Wire Wire Line
-	7350 4350 7100 4350
-Connection ~ 7100 4350
+	5850 2950 5850 3200
 $EndSCHEMATC
