File: Cube/PCB/Block Layers Catodes.sch (KiCad schematic (older format))
At the start: 10 parts

Commit message: Update
Update
Parts:
- gave numbers to parts that had none: 10
Connections:
- net +5V: no longer U8.10 (~SRCLR)
- new net ~SRCLR: U8.10 (~SRCLR)
Other:
- moved on the sheet: C10, Q1, Q2, Q3, Q4, Q5, Q6, Q7, Q8, U8

Commit message: Update project
Remove a image corrupted -_-
Parts:
- C10: footprint (none) -> alex-library:C-P_5.08-L_7.5-H_6-P_2.5
- U8: footprint (none) -> alex-library:DIP-16_W7.62mm_LongPads
Changed lines of the file:
@@
 $Descr A4 11693 8268
 encoding utf-8
-Sheet 10 12
+Sheet 12 12
 Title ""
 Date ""
@@
 F 0 "U8" H 3000 5050 60  0000 C CNN
 F 1 "SN74HC595" H 3200 3950 60  0000 C CNN
-F 2 "" H 3550 4400 60  0001 C CNN
+F 2 "alex-library:DIP-16_W7.62mm_LongPads" H 3550 4400 60  0001 C CNN
 F 3 "" H 3550 4400 60  0001 C CNN
 	1    3200 4500
@@
 F 0 "C10" H 2975 3350 50  0000 L CNN
 F 1 "100nF" H 2975 3150 50  0000 L CNN
-F 2 "" H 2988 3100 50  0001 C CNN
+F 2 "alex-library:C-P_5.08-L_7.5-H_6-P_2.5" H 2988 3100 50  0001 C CNN
 F 3 "" H 2950 3250 50  0001 C CNN
 	1    2950 3250
@@
 $EndComp
 $Comp
-L +5V #PWR40
+L +5V #PWR054
 U 1 1 5B243FAE
 P 2950 2950
-F 0 "#PWR40" H 2950 2800 50  0001 C CNN
+F 0 "#PWR054" H 2950 2800 50  0001 C CNN
 F 1 "+5V" H 2950 3090 50  0000 C CNN
 F 2 "" H 2950 2950 50  0001 C CNN
@@
 $EndComp
 $Comp
-L GND #PWR41
+L GND #PWR055
 U 1 1 5B243FAF
 P 2950 3550
-F 0 "#PWR41" H 2950 3300 50  0001 C CNN
+F 0 "#PWR055" H 2950 3300 50  0001 C CNN
 F 1 "GND" H 2950 3400 50  0000 C CNN
 F 2 "" H 2950 3550 50  0001 C CNN
@@
 $EndComp
 $Comp
-L GND #PWR39
+L GND #PWR056
 U 1 1 5B243FB0
 P 2600 4250
-F 0 "#PWR39" H 2600 4000 50  0001 C CNN
+F 0 "#PWR056" H 2600 4000 50  0001 C CNN
 F 1 "GND" H 2600 4100 50  0000 C CNN
 F 2 "" H 2600 4250 50  0001 C CNN
@@
 $EndComp
 $Comp
-L GND #PWR38
+L GND #PWR057
 U 1 1 5B243FB2
 P 2300 4850
-F 0 "#PWR38" H 2300 4600 50  0001 C CNN
+F 0 "#PWR057" H 2300 4600 50  0001 C CNN
 F 1 "GND" H 2300 4700 50  0000 C CNN
 F 2 "" H 2300 4850 50  0001 C CNN
@@
 $EndComp
 $Comp
-L GND #PWR42
+L GND #PWR058
 U 1 1 5B24429E
 P 4300 4050
-F 0 "#PWR42" H 4300 3800 50  0001 C CNN
+F 0 "#PWR058" H 4300 3800 50  0001 C CNN
 F 1 "GND" H 4300 3900 50  0000 C CNN
 F 2 "" H 4300 4050 50  0001 C CNN
@@
 $EndComp
 $Comp
-L GND #PWR43
+L GND #PWR059
 U 1 1 5B24438F
 P 5200 4050
-F 0 "#PWR43" H 5200 3800 50  0001 C CNN
+F 0 "#PWR059" H 5200 3800 50  0001 C CNN
 F 1 "GND" H 5200 3900 50  0000 C CNN
 F 2 "" H 5200 4050 50  0001 C CNN
@@
 $EndComp
 $Comp
-L GND #PWR44
+L GND #PWR060
 U 1 1 5B244429
 P 6100 4050
-F 0 "#PWR44" H 6100 3800 50  0001 C CNN
+F 0 "#PWR060" H 6100 3800 50  0001 C CNN
 F 1 "GND" H 6100 3900 50  0000 C CNN
 F 2 "" H 6100 4050 50  0001 C CNN
@@
 $EndComp
 $Comp
-L GND #PWR45
+L GND #PWR061
 U 1 1 5B244439
 P 7000 4050
-F 0 "#PWR45" H 7000 3800 50  0001 C CNN
+F 0 "#PWR061" H 7000 3800 50  0001 C CNN
 F 1 "GND" H 7000 3900 50  0000 C CNN
 F 2 "" H 7000 4050 50  0001 C CNN
@@
 $EndComp
 $Comp
-L GND #PWR46
+L GND #PWR062
 U 1 1 5B244551
 P 7900 4050
-F 0 "#PWR46" H 7900 3800 50  0001 C CNN
+F 0 "#PWR062" H 7900 3800 50  0001 C CNN
 F 1 "GND" H 7900 3900 50  0000 C CNN
 F 2 "" H 7900 4050 50  0001 C CNN
@@
 $EndComp
 $Comp
-L GND #PWR47
+L GND #PWR063
 U 1 1 5B244561
 P 8800 4050
-F 0 "#PWR47" H 8800 3800 50  0001 C CNN
+F 0 "#PWR063" H 8800 3800 50  0001 C CNN
 F 1 "GND" H 8800 3900 50  0000 C CNN
 F 2 "" H 8800 4050 50  0001 C CNN
@@
 $EndComp
 $Comp
-L GND #PWR48
+L GND #PWR064
 U 1 1 5B244571
 P 9700 4050
-F 0 "#PWR48" H 9700 3800 50  0001 C CNN
+F 0 "#PWR064" H 9700 3800 50  0001 C CNN
 F 1 "GND" H 9700 3900 50  0000 C CNN
 F 2 "" H 9700 4050 50  0001 C CNN
@@
 $EndComp
 $Comp
-L GND #PWR49
+L GND #PWR065
 U 1 1 5B244581
 P 10600 4050
-F 0 "#PWR49" H 10600 3800 50  0001 C CNN
+F 0 "#PWR065" H 10600 3800 50  0001 C CNN
 F 1 "GND" H 10600 3900 50  0000 C CNN
 F 2 "" H 10600 4050 50  0001 C CNN

Commit message: Update project
Update
Parts:
- Q1, Q2, Q3, Q4, Q5, Q6, Q7, Q8: footprint TO_SOT_Packages_THT:TO-92_Molded_Narrow -> alex-library:TO-92_Inline_Narrow_Oval
- renumbered C10 to C12, U8 to U10
Changed lines of the file:
@@
 encoding utf-8
 Sheet 12 12
-Title ""
-Date ""
-Rev ""
-Comp ""
+Title "Logique de commande Cube 8x8x8 512 Leds"
+Date "2018-06-21"
+Rev "1"
+Comp "FabLab19"
 Comment1 ""
 Comment2 ""
@@
 $EndDescr
 $Comp
-L SN74HC595 U8
+L SN74HC595 U10
 U 1 1 5B243FAC
 P 3200 4500
-F 0 "U8" H 3000 5050 60  0000 C CNN
+F 0 "U10" H 3000 5050 60  0000 C CNN
 F 1 "SN74HC595" H 3200 3950 60  0000 C CNN
 F 2 "alex-library:DIP-16_W7.62mm_LongPads" H 3550 4400 60  0001 C CNN
@@
 $EndComp
 $Comp
-L C C10
+L C C12
 U 1 1 5B243FAD
 P 2950 3250
-F 0 "C10" H 2975 3350 50  0000 L CNN
+F 0 "C12" H 2975 3350 50  0000 L CNN
 F 1 "100nF" H 2975 3150 50  0000 L CNN
 F 2 "alex-library:C-P_5.08-L_7.5-H_6-P_2.5" H 2988 3100 50  0001 C CNN
@@
 F 0 "Q1" H 4400 3825 50  0000 L CNN
 F 1 "PN2222A" H 4400 3750 50  0000 L CNN
-F 2 "TO_SOT_Packages_THT:TO-92_Molded_Narrow" H 4400 3675 50  0001 L CIN
+F 2 "alex-library:TO-92_Inline_Narrow_Oval" H 4400 3675 50  0001 L CIN
 F 3 "" H 4200 3750 50  0001 L CNN
 	1    4200 3750
@@
 F 0 "Q2" H 5300 3825 50  0000 L CNN
 F 1 "PN2222A" H 5300 3750 50  0000 L CNN
-F 2 "TO_SOT_Packages_THT:TO-92_Molded_Narrow" H 5300 3675 50  0001 L CIN
+F 2 "alex-library:TO-92_Inline_Narrow_Oval" H 5300 3675 50  0001 L CIN
 F 3 "" H 5100 3750 50  0001 L CNN
 	1    5100 3750
@@
 F 0 "Q3" H 6200 3825 50  0000 L CNN
 F 1 "PN2222A" H 6200 3750 50  0000 L CNN
-F 2 "TO_SOT_Packages_THT:TO-92_Molded_Narrow" H 6200 3675 50  0001 L CIN
+F 2 "alex-library:TO-92_Inline_Narrow_Oval" H 6200 3675 50  0001 L CIN
 F 3 "" H 6000 3750 50  0001 L CNN
 	1    6000 3750
@@
 F 0 "Q4" H 7100 3825 50  0000 L CNN
 F 1 "PN2222A" H 7100 3750 50  0000 L CNN
-F 2 "TO_SOT_Packages_THT:TO-92_Molded_Narrow" H 7100 3675 50  0001 L CIN
+F 2 "alex-library:TO-92_Inline_Narrow_Oval" H 7100 3675 50  0001 L CIN
 F 3 "" H 6900 3750 50  0001 L CNN
 	1    6900 3750
@@
 F 0 "Q5" H 8000 3825 50  0000 L CNN
 F 1 "PN2222A" H 8000 3750 50  0000 L CNN
-F 2 "TO_SOT_Packages_THT:TO-92_Molded_Narrow" H 8000 3675 50  0001 L CIN
+F 2 "alex-library:TO-92_Inline_Narrow_Oval" H 8000 3675 50  0001 L CIN
 F 3 "" H 7800 3750 50  0001 L CNN
 	1    7800 3750
@@
 F 0 "Q6" H 8900 3825 50  0000 L CNN
 F 1 "PN2222A" H 8900 3750 50  0000 L CNN
-F 2 "TO_SOT_Packages_THT:TO-92_Molded_Narrow" H 8900 3675 50  0001 L CIN
+F 2 "alex-library:TO-92_Inline_Narrow_Oval" H 8900 3675 50  0001 L CIN
 F 3 "" H 8700 3750 50  0001 L CNN
 	1    8700 3750
@@
 F 0 "Q7" H 9800 3825 50  0000 L CNN
 F 1 "PN2222A" H 9800 3750 50  0000 L CNN
-F 2 "TO_SOT_Packages_THT:TO-92_Molded_Narrow" H 9800 3675 50  0001 L CIN
+F 2 "alex-library:TO-92_Inline_Narrow_Oval" H 9800 3675 50  0001 L CIN
 F 3 "" H 9600 3750 50  0001 L CNN
 	1    9600 3750
@@
 F 0 "Q8" H 10700 3825 50  0000 L CNN
 F 1 "PN2222A" H 10700 3750 50  0000 L CNN
-F 2 "TO_SOT_Packages_THT:TO-92_Molded_Narrow" H 10700 3675 50  0001 L CIN
+F 2 "alex-library:TO-92_Inline_Narrow_Oval" H 10700 3675 50  0001 L CIN
 F 3 "" H 10500 3750 50  0001 L CNN
 	1    10500 3750

Commit message: Update
Update
Changed lines of the file:
@@
 	2300 4800 2300 4850
-Wire Wire Line
-	1400 4600 2750 4600
 Wire Wire Line
 	1400 4700 2750 4700
@@
 Wire Wire Line
 	1800 4500 2750 4500
+Wire Wire Line
+	2750 4600 1400 4600
 $EndSCHEMATC

Commit message: Update
Update
Add New restistor in Base Q1, Q2, Q3, Q4, Q5, Q6, Q7, Q8
New version PCB
New rename components
Parts:
- added R66, R67, R68, R69, R70, R71, R72, R73: 1,1K, alex-library:R_Axial_Long6.3mm_Dia2.5mm_Pas15.24mm_Horizontal, symbol R
Connections:
- net at U10.1 (QB): now also R67.1; no longer Q2.2 (B)
- net at U10.15 (QA): now also R66.1; no longer Q1.2 (B)
- net at U10.2 (QC): now also R68.1; no longer Q3.2 (B)
- net at U10.3 (QD): now also R69.1; no longer Q4.2 (B)
- net at U10.4 (QE): now also R70.1; no longer Q5.2 (B)
- net at U10.5 (QF): now also R71.1; no longer Q6.2 (B)
- net at U10.6 (QG): now also R72.1; no longer Q7.2 (B)
- net at U10.7 (QH): now also R73.1; no longer Q8.2 (B)
- new net: Q1.2 (B), R66.2
- new net: Q2.2 (B), R67.2
- new net: Q3.2 (B), R68.2
- new net: Q4.2 (B), R69.2
- new net: Q5.2 (B), R70.2
- new net: Q6.2 (B), R71.2
- new net: Q7.2 (B), R72.2
- new net: Q8.2 (B), R73.2
