File: Cube/PCB/Block Row Anode 1.sch (KiCad schematic (older format))
At the start: 10 parts, among them U4 SN74HC595

Commit message: Update
Update
Parts:
- removed C6: 100nF, symbol C
- removed R20, R21, R22, R23, R24, R25, R26, R27: R, symbol R
- removed U4: SN74HC595, symbol SN74HC595
- added C4: 100nF, symbol C
- added R10, R11, R4, R5, R6, R7, R8, R9: R, symbol R
- added U2: SN74HC595, symbol SN74HC595
Connections:
- net +5V: now also C4.1, U2.16 (VCC)
- net GND: now also C4.2, U2.13 (~OE), U2.8 (GND)
- net RCLK: now also U2.12 (RCLK)
- net R_QA: now also R4.1
- net R_QB: now also R5.1
- net R_QC: now also R6.1
- net R_QD: now also R7.1
- net R_QE: now also R8.1
- net R_QF: now also R9.1
- net R_QG: now also R10.1
- net R_QH: now also R11.1
- net R_QH': now also U2.9 (QH')
- net SER: now also U2.14 (SER)
- net SRCLK: now also U2.11 (SRCLK)
- net ~SRCLR: now also U2.10 (~SRCLR)
- new net: R10.2, U2.6 (QG)
- new net: R5.2, U2.1 (QB)
- new net: R4.2, U2.15 (QA)
- new net: R6.2, U2.2 (QC)
- new net: R7.2, U2.3 (QD)
- new net: R8.2, U2.4 (QE)
- new net: R9.2, U2.5 (QF)
- new net: R11.2, U2.7 (QH)
Changed lines of the file:
@@
 $Descr A4 11693 8268
 encoding utf-8
-Sheet 6 12
+Sheet 4 12
 Title ""
 Date ""
@@
 $EndDescr
 $Comp
-L SN74HC595 U4
-U 1 1 5B234BDC
+L SN74HC595 U2
+U 1 1 5B247E1E
 P 4900 3650
-F 0 "U4" H 4700 4200 60  0000 C CNN
+F 0 "U2" H 4700 4200 60  0000 C CNN
 F 1 "SN74HC595" H 4900 3100 60  0000 C CNN
 F 2 "" H 5250 3550 60  0001 C CNN
@@
 $EndComp
 $Comp
-L C C6
-U 1 1 5B234BDD
+L C C4
+U 1 1 5B247E2A
 P 3750 3000
-F 0 "C6" H 3775 3100 50  0000 L CNN
+F 0 "C4" H 3775 3100 50  0000 L CNN
 F 1 "100nF" H 3775 2900 50  0000 L CNN
 F 2 "" H 3788 2850 50  0001 C CNN
@@
 $EndComp
 $Comp
-L +5V #PWR22
-U 1 1 5B234BDE
+L +5V #PWR14
+U 1 1 5B247E2C
 P 3750 2700
-F 0 "#PWR22" H 3750 2550 50  0001 C CNN
+F 0 "#PWR14" H 3750 2550 50  0001 C CNN
 F 1 "+5V" H 3750 2840 50  0000 C CNN
 F 2 "" H 3750 2700 50  0001 C CNN
@@
 $EndComp
 $Comp
-L GND #PWR23
-U 1 1 5B234BDF
+L GND #PWR15
+U 1 1 5B247E39
 P 3750 3300
-F 0 "#PWR23" H 3750 3050 50  0001 C CNN
+F 0 "#PWR15" H 3750 3050 50  0001 C CNN
 F 1 "GND" H 3750 3150 50  0000 C CNN
 F 2 "" H 3750 3300 50  0001 C CNN
@@
 $EndComp
 $Comp
-L GND #PWR25
-U 1 1 5B234BE0
+L GND #PWR17
+U 1 1 5B2236C5
 P 4300 3400
-F 0 "#PWR25" H 4300 3150 50  0001 C CNN
+F 0 "#PWR17" H 4300 3150 50  0001 C CNN
 F 1 "GND" H 4300 3250 50  0000 C CNN
 F 2 "" H 4300 3400 50  0001 C CNN
@@
 $EndComp
 $Comp
-L GND #PWR24
-U 1 1 5B234BE1
+L GND #PWR16
+U 1 1 5B247E4A
 P 4000 4000
-F 0 "#PWR24" H 4000 3750 50  0001 C CNN
+F 0 "#PWR16" H 4000 3750 50  0001 C CNN
 F 1 "GND" H 4000 3850 50  0000 C CNN
 F 2 "" H 4000 4000 50  0001 C CNN
@@
 R_QH'
 $Comp
-L R R20
-U 1 1 5B234BE2
+L R R4
+U 1 1 5B247E50
 P 5650 3250
-F 0 "R20" V 5730 3250 50  0000 C CNN
+F 0 "R4" V 5730 3250 50  0000 C CNN
 F 1 "R" V 5650 3250 50  0000 C CNN
 F 2 "" V 5580 3250 50  0001 C CNN
@@
 $EndComp
 $Comp
-L R R21
-U 1 1 5B234BE3
+L R R5
+U 1 1 5B247E5B
 P 5900 3350
-F 0 "R21" V 5980 3350 50  0000 C CNN
+F 0 "R5" V 5980 3350 50  0000 C CNN
 F 1 "R" V 5900 3350 50  0000 C CNN
 F 2 "" V 5830 3350 50  0001 C CNN
@@
 $EndComp
 $Comp
-L R R22
-U 1 1 5B234BE4
+L R R6
+U 1 1 5B247E61
 P 6150 3450
-F 0 "R22" V 6230 3450 50  0000 C CNN
+F 0 "R6" V 6230 3450 50  0000 C CNN
 F 1 "R" V 6150 3450 50  0000 C CNN
 F 2 "" V 6080 3450 50  0001 C CNN
@@
 $EndComp
 $Comp
-L R R23
-U 1 1 5B234BE5
+L R R7
+U 1 1 5B247E67
 P 6400 3550
-F 0 "R23" V 6480 3550 50  0000 C CNN
+F 0 "R7" V 6480 3550 50  0000 C CNN
 F 1 "R" V 6400 3550 50  0000 C CNN
 F 2 "" V 6330 3550 50  0001 C CNN
@@
 $EndComp
 $Comp
-L R R24
-U 1 1 5B234BE6
+L R R8
+U 1 1 5B247E70
 P 6650 3650
-F 0 "R24" V 6730 3650 50  0000 C CNN
+F 0 "R8" V 6730 3650 50  0000 C CNN
 F 1 "R" V 6650 3650 50  0000 C CNN
 F 2 "" V 6580 3650 50  0001 C CNN
@@
 $EndComp
 $Comp
-L R R25
-U 1 1 5B234BE7
+L R R9
+U 1 1 5B247E78
 P 6900 3750
-F 0 "R25" V 6980 3750 50  0000 C CNN
+F 0 "R9" V 6980 3750 50  0000 C CNN
 F 1 "R" V 6900 3750 50  0000 C CNN
 F 2 "" V 6830 3750 50  0001 C CNN
@@
 $EndComp
 $Comp
-L R R26
-U 1 1 5B234BE8
+L R R10
+U 1 1 5B223B39
 P 7150 3850
-F 0 "R26" V 7230 3850 50  0000 C CNN
+F 0 "R10" V 7230 3850 50  0000 C CNN
 F 1 "R" V 7150 3850 50  0000 C CNN
 F 2 "" V 7080 3850 50  0001 C CNN
@@
 	5350 3850 7000 3850
 $Comp
-L R R27
-U 1 1 5B234BE9
+L R R11
+U 1 1 5B247E80
 P 7400 3950
-F 0 "R27" V 7480 3950 50  0000 C CNN
+F 0 "R11" V 7480 3950 50  0000 C CNN
 F 1 "R" V 7400 3950 50  0000 C CNN
 F 2 "" V 7330 3950 50  0001 C CNN

Commit message: Update project
Remove a image corrupted -_-
Parts:
- C4: footprint (none) -> alex-library:C-P_5.08-L_7.5-H_6-P_2.5
- R10, R11, R4, R5, R6, R7, R8, R9: footprint (none) -> alex-library:R_Axial_Long6.3mm_Dia2.5mm_Pas15.24mm_Horizontal
- U2: footprint (none) -> alex-library:DIP-16_W7.62mm_LongPads
Changed lines of the file:
@@
 F 0 "U2" H 4700 4200 60  0000 C CNN
 F 1 "SN74HC595" H 4900 3100 60  0000 C CNN
-F 2 "" H 5250 3550 60  0001 C CNN
+F 2 "alex-library:DIP-16_W7.62mm_LongPads" H 5250 3550 60  0001 C CNN
 F 3 "" H 5250 3550 60  0001 C CNN
 	1    4900 3650
@@
 F 0 "C4" H 3775 3100 50  0000 L CNN
 F 1 "100nF" H 3775 2900 50  0000 L CNN
-F 2 "" H 3788 2850 50  0001 C CNN
+F 2 "alex-library:C-P_5.08-L_7.5-H_6-P_2.5" H 3788 2850 50  0001 C CNN
 F 3 "" H 3750 3000 50  0001 C CNN
 	1    3750 3000
@@
 $EndComp
 $Comp
-L +5V #PWR14
+L +5V #PWR022
 U 1 1 5B247E2C
 P 3750 2700
-F 0 "#PWR14" H 3750 2550 50  0001 C CNN
+F 0 "#PWR022" H 3750 2550 50  0001 C CNN
 F 1 "+5V" H 3750 2840 50  0000 C CNN
 F 2 "" H 3750 2700 50  0001 C CNN
@@
 $EndComp
 $Comp
-L GND #PWR15
+L GND #PWR023
 U 1 1 5B247E39
 P 3750 3300
-F 0 "#PWR15" H 3750 3050 50  0001 C CNN
+F 0 "#PWR023" H 3750 3050 50  0001 C CNN
 F 1 "GND" H 3750 3150 50  0000 C CNN
 F 2 "" H 3750 3300 50  0001 C CNN
@@
 $EndComp
 $Comp
-L GND #PWR17
+L GND #PWR024
 U 1 1 5B2236C5
 P 4300 3400
-F 0 "#PWR17" H 4300 3150 50  0001 C CNN
+F 0 "#PWR024" H 4300 3150 50  0001 C CNN
 F 1 "GND" H 4300 3250 50  0000 C CNN
 F 2 "" H 4300 3400 50  0001 C CNN
@@
 $EndComp
 $Comp
-L GND #PWR16
+L GND #PWR025
 U 1 1 5B247E4A
 P 4000 4000
-F 0 "#PWR16" H 4000 3750 50  0001 C CNN
+F 0 "#PWR025" H 4000 3750 50  0001 C CNN
 F 1 "GND" H 4000 3850 50  0000 C CNN
 F 2 "" H 4000 4000 50  0001 C CNN
@@
 F 0 "R4" V 5730 3250 50  0000 C CNN
 F 1 "R" V 5650 3250 50  0000 C CNN
-F 2 "" V 5580 3250 50  0001 C CNN
+F 2 "alex-library:R_Axial_Long6.3mm_Dia2.5mm_Pas15.24mm_Horizontal" V 5580 3250 50  0001 C CNN
 F 3 "" H 5650 3250 50  0001 C CNN
 	1    5650 3250
@@
 F 0 "R5" V 5980 3350 50  0000 C CNN
 F 1 "R" V 5900 3350 50  0000 C CNN
-F 2 "" V 5830 3350 50  0001 C CNN
+F 2 "alex-library:R_Axial_Long6.3mm_Dia2.5mm_Pas15.24mm_Horizontal" V 5830 3350 50  0001 C CNN
 F 3 "" H 5900 3350 50  0001 C CNN
 	1    5900 3350
@@
 F 0 "R6" V 6230 3450 50  0000 C CNN
 F 1 "R" V 6150 3450 50  0000 C CNN
-F 2 "" V 6080 3450 50  0001 C CNN
+F 2 "alex-library:R_Axial_Long6.3mm_Dia2.5mm_Pas15.24mm_Horizontal" V 6080 3450 50  0001 C CNN
 F 3 "" H 6150 3450 50  0001 C CNN
 	1    6150 3450
@@
 F 0 "R7" V 6480 3550 50  0000 C CNN
 F 1 "R" V 6400 3550 50  0000 C CNN
-F 2 "" V 6330 3550 50  0001 C CNN
+F 2 "alex-library:R_Axial_Long6.3mm_Dia2.5mm_Pas15.24mm_Horizontal" V 6330 3550 50  0001 C CNN
 F 3 "" H 6400 3550 50  0001 C CNN
 	1    6400 3550
@@
 F 0 "R8" V 6730 3650 50  0000 C CNN
 F 1 "R" V 6650 3650 50  0000 C CNN
-F 2 "" V 6580 3650 50  0001 C CNN
+F 2 "alex-library:R_Axial_Long6.3mm_Dia2.5mm_Pas15.24mm_Horizontal" V 6580 3650 50  0001 C CNN
 F 3 "" H 6650 3650 50  0001 C CNN
 	1    6650 3650
@@
 F 0 "R9" V 6980 3750 50  0000 C CNN
 F 1 "R" V 6900 3750 50  0000 C CNN
-F 2 "" V 6830 3750 50  0001 C CNN
+F 2 "alex-library:R_Axial_Long6.3mm_Dia2.5mm_Pas15.24mm_Horizontal" V 6830 3750 50  0001 C CNN
 F 3 "" H 6900 3750 50  0001 C CNN
 	1    6900 3750
@@
 F 0 "R10" V 7230 3850 50  0000 C CNN
 F 1 "R" V 7150 3850 50  0000 C CNN
-F 2 "" V 7080 3850 50  0001 C CNN
+F 2 "alex-library:R_Axial_Long6.3mm_Dia2.5mm_Pas15.24mm_Horizontal" V 7080 3850 50  0001 C CNN
 F 3 "" H 7150 3850 50  0001 C CNN
 	1    7150 3850
@@
 F 0 "R11" V 7480 3950 50  0000 C CNN
 F 1 "R" V 7400 3950 50  0000 C CNN
-F 2 "" V 7330 3950 50  0001 C CNN
+F 2 "alex-library:R_Axial_Long6.3mm_Dia2.5mm_Pas15.24mm_Horizontal" V 7330 3950 50  0001 C CNN
 F 3 "" H 7400 3950 50  0001 C CNN
 	1    7400 3950

Commit message: Update
Update
Add New restistor in Base Q1, Q2, Q3, Q4, Q5, Q6, Q7, Q8
New version PCB
New rename components
Parts:
- renumbered R4 to R2, R5 to R3, R6 to R4, R7 to R5, R8 to R6, R9 to R7, R10 to R8, R11 to R9
Changed lines of the file:
@@
 R_QH'
 $Comp
-L R R4
+L R R2
 U 1 1 5B247E50
 P 5650 3250
-F 0 "R4" V 5730 3250 50  0000 C CNN
+F 0 "R2" V 5730 3250 50  0000 C CNN
 F 1 "R" V 5650 3250 50  0000 C CNN
 F 2 "alex-library:R_Axial_Long6.3mm_Dia2.5mm_Pas15.24mm_Horizontal" V 5580 3250 50  0001 C CNN
@@
 $EndComp
 $Comp
-L R R5
+L R R3
 U 1 1 5B247E5B
 P 5900 3350
-F 0 "R5" V 5980 3350 50  0000 C CNN
+F 0 "R3" V 5980 3350 50  0000 C CNN
 F 1 "R" V 5900 3350 50  0000 C CNN
 F 2 "alex-library:R_Axial_Long6.3mm_Dia2.5mm_Pas15.24mm_Horizontal" V 5830 3350 50  0001 C CNN
@@
 $EndComp
 $Comp
-L R R6
+L R R4
 U 1 1 5B247E61
 P 6150 3450
-F 0 "R6" V 6230 3450 50  0000 C CNN
+F 0 "R4" V 6230 3450 50  0000 C CNN
 F 1 "R" V 6150 3450 50  0000 C CNN
 F 2 "alex-library:R_Axial_Long6.3mm_Dia2.5mm_Pas15.24mm_Horizontal" V 6080 3450 50  0001 C CNN
@@
 $EndComp
 $Comp
-L R R7
+L R R5
 U 1 1 5B247E67
 P 6400 3550
-F 0 "R7" V 6480 3550 50  0000 C CNN
+F 0 "R5" V 6480 3550 50  0000 C CNN
 F 1 "R" V 6400 3550 50  0000 C CNN
 F 2 "alex-library:R_Axial_Long6.3mm_Dia2.5mm_Pas15.24mm_Horizontal" V 6330 3550 50  0001 C CNN
@@
 $EndComp
 $Comp
-L R R8
+L R R6
 U 1 1 5B247E70
 P 6650 3650
-F 0 "R8" V 6730 3650 50  0000 C CNN
+F 0 "R6" V 6730 3650 50  0000 C CNN
 F 1 "R" V 6650 3650 50  0000 C CNN
 F 2 "alex-library:R_Axial_Long6.3mm_Dia2.5mm_Pas15.24mm_Horizontal" V 6580 3650 50  0001 C CNN
@@
 $EndComp
 $Comp
-L R R9
+L R R7
 U 1 1 5B247E78
 P 6900 3750
-F 0 "R9" V 6980 3750 50  0000 C CNN
+F 0 "R7" V 6980 3750 50  0000 C CNN
 F 1 "R" V 6900 3750 50  0000 C CNN
 F 2 "alex-library:R_Axial_Long6.3mm_Dia2.5mm_Pas15.24mm_Horizontal" V 6830 3750 50  0001 C CNN
@@
 $EndComp
 $Comp
-L R R10
+L R R8
 U 1 1 5B223B39
 P 7150 3850
-F 0 "R10" V 7230 3850 50  0000 C CNN
+F 0 "R8" V 7230 3850 50  0000 C CNN
 F 1 "R" V 7150 3850 50  0000 C CNN
 F 2 "alex-library:R_Axial_Long6.3mm_Dia2.5mm_Pas15.24mm_Horizontal" V 7080 3850 50  0001 C CNN
@@
 	5350 3850 7000 3850
 $Comp
-L R R11
+L R R9
 U 1 1 5B247E80
 P 7400 3950
-F 0 "R11" V 7480 3950 50  0000 C CNN
+F 0 "R9" V 7480 3950 50  0000 C CNN
 F 1 "R" V 7400 3950 50  0000 C CNN
 F 2 "alex-library:R_Axial_Long6.3mm_Dia2.5mm_Pas15.24mm_Horizontal" V 7330 3950 50  0001 C CNN
