File: Cube/PCB/Block Row Anode 5.sch (KiCad schematic (older format))
At the start: 10 parts, among them U4 SN74HC595

Commit message: Update project
Remove a image corrupted -_-
Parts:
- C6: footprint (none) -> alex-library:C-P_5.08-L_7.5-H_6-P_2.5
- R20, R21, R22, R23, R24, R25, R26, R27: footprint (none) -> alex-library:R_Axial_Long6.3mm_Dia2.5mm_Pas15.24mm_Horizontal
- U4: footprint (none) -> alex-library:DIP-16_W7.62mm_LongPads
Changed lines of the file:
@@
 F 0 "U4" H 4700 4200 60  0000 C CNN
 F 1 "SN74HC595" H 4900 3100 60  0000 C CNN
-F 2 "" H 5250 3550 60  0001 C CNN
+F 2 "alex-library:DIP-16_W7.62mm_LongPads" H 5250 3550 60  0001 C CNN
 F 3 "" H 5250 3550 60  0001 C CNN
 	1    4900 3650
@@
 F 0 "C6" H 3775 3100 50  0000 L CNN
 F 1 "100nF" H 3775 2900 50  0000 L CNN
-F 2 "" H 3788 2850 50  0001 C CNN
+F 2 "alex-library:C-P_5.08-L_7.5-H_6-P_2.5" H 3788 2850 50  0001 C CNN
 F 3 "" H 3750 3000 50  0001 C CNN
 	1    3750 3000
@@
 $EndComp
 $Comp
-L +5V #PWR22
+L +5V #PWR030
 U 1 1 5B234BDE
 P 3750 2700
-F 0 "#PWR22" H 3750 2550 50  0001 C CNN
+F 0 "#PWR030" H 3750 2550 50  0001 C CNN
 F 1 "+5V" H 3750 2840 50  0000 C CNN
 F 2 "" H 3750 2700 50  0001 C CNN
@@
 $EndComp
 $Comp
-L GND #PWR23
+L GND #PWR031
 U 1 1 5B234BDF
 P 3750 3300
-F 0 "#PWR23" H 3750 3050 50  0001 C CNN
+F 0 "#PWR031" H 3750 3050 50  0001 C CNN
 F 1 "GND" H 3750 3150 50  0000 C CNN
 F 2 "" H 3750 3300 50  0001 C CNN
@@
 $EndComp
 $Comp
-L GND #PWR25
+L GND #PWR032
 U 1 1 5B234BE0
 P 4300 3400
-F 0 "#PWR25" H 4300 3150 50  0001 C CNN
+F 0 "#PWR032" H 4300 3150 50  0001 C CNN
 F 1 "GND" H 4300 3250 50  0000 C CNN
 F 2 "" H 4300 3400 50  0001 C CNN
@@
 $EndComp
 $Comp
-L GND #PWR24
+L GND #PWR033
 U 1 1 5B234BE1
 P 4000 4000
-F 0 "#PWR24" H 4000 3750 50  0001 C CNN
+F 0 "#PWR033" H 4000 3750 50  0001 C CNN
 F 1 "GND" H 4000 3850 50  0000 C CNN
 F 2 "" H 4000 4000 50  0001 C CNN
@@
 F 0 "R20" V 5730 3250 50  0000 C CNN
 F 1 "R" V 5650 3250 50  0000 C CNN
-F 2 "" V 5580 3250 50  0001 C CNN
+F 2 "alex-library:R_Axial_Long6.3mm_Dia2.5mm_Pas15.24mm_Horizontal" V 5580 3250 50  0001 C CNN
 F 3 "" H 5650 3250 50  0001 C CNN
 	1    5650 3250
@@
 F 0 "R21" V 5980 3350 50  0000 C CNN
 F 1 "R" V 5900 3350 50  0000 C CNN
-F 2 "" V 5830 3350 50  0001 C CNN
+F 2 "alex-library:R_Axial_Long6.3mm_Dia2.5mm_Pas15.24mm_Horizontal" V 5830 3350 50  0001 C CNN
 F 3 "" H 5900 3350 50  0001 C CNN
 	1    5900 3350
@@
 F 0 "R22" V 6230 3450 50  0000 C CNN
 F 1 "R" V 6150 3450 50  0000 C CNN
-F 2 "" V 6080 3450 50  0001 C CNN
+F 2 "alex-library:R_Axial_Long6.3mm_Dia2.5mm_Pas15.24mm_Horizontal" V 6080 3450 50  0001 C CNN
 F 3 "" H 6150 3450 50  0001 C CNN
 	1    6150 3450
@@
 F 0 "R23" V 6480 3550 50  0000 C CNN
 F 1 "R" V 6400 3550 50  0000 C CNN
-F 2 "" V 6330 3550 50  0001 C CNN
+F 2 "alex-library:R_Axial_Long6.3mm_Dia2.5mm_Pas15.24mm_Horizontal" V 6330 3550 50  0001 C CNN
 F 3 "" H 6400 3550 50  0001 C CNN
 	1    6400 3550
@@
 F 0 "R24" V 6730 3650 50  0000 C CNN
 F 1 "R" V 6650 3650 50  0000 C CNN
-F 2 "" V 6580 3650 50  0001 C CNN
+F 2 "alex-library:R_Axial_Long6.3mm_Dia2.5mm_Pas15.24mm_Horizontal" V 6580 3650 50  0001 C CNN
 F 3 "" H 6650 3650 50  0001 C CNN
 	1    6650 3650
@@
 F 0 "R25" V 6980 3750 50  0000 C CNN
 F 1 "R" V 6900 3750 50  0000 C CNN
-F 2 "" V 6830 3750 50  0001 C CNN
+F 2 "alex-library:R_Axial_Long6.3mm_Dia2.5mm_Pas15.24mm_Horizontal" V 6830 3750 50  0001 C CNN
 F 3 "" H 6900 3750 50  0001 C CNN
 	1    6900 3750
@@
 F 0 "R26" V 7230 3850 50  0000 C CNN
 F 1 "R" V 7150 3850 50  0000 C CNN
-F 2 "" V 7080 3850 50  0001 C CNN
+F 2 "alex-library:R_Axial_Long6.3mm_Dia2.5mm_Pas15.24mm_Horizontal" V 7080 3850 50  0001 C CNN
 F 3 "" H 7150 3850 50  0001 C CNN
 	1    7150 3850
@@
 F 0 "R27" V 7480 3950 50  0000 C CNN
 F 1 "R" V 7400 3950 50  0000 C CNN
-F 2 "" V 7330 3950 50  0001 C CNN
+F 2 "alex-library:R_Axial_Long6.3mm_Dia2.5mm_Pas15.24mm_Horizontal" V 7330 3950 50  0001 C CNN
 F 3 "" H 7400 3950 50  0001 C CNN
 	1    7400 3950

Commit message: Update
Update
Add New restistor in Base Q1, Q2, Q3, Q4, Q5, Q6, Q7, Q8
New version PCB
New rename components
Parts:
- renumbered R20 to R18, R21 to R19, R22 to R20, R23 to R21, R24 to R22, R25 to R23, R26 to R24, R27 to R25
Changed lines of the file:
@@
 R_QH'
 $Comp
-L R R20
+L R R18
 U 1 1 5B234BE2
 P 5650 3250
-F 0 "R20" V 5730 3250 50  0000 C CNN
+F 0 "R18" V 5730 3250 50  0000 C CNN
 F 1 "R" V 5650 3250 50  0000 C CNN
 F 2 "alex-library:R_Axial_Long6.3mm_Dia2.5mm_Pas15.24mm_Horizontal" V 5580 3250 50  0001 C CNN
@@
 $EndComp
 $Comp
-L R R21
+L R R19
 U 1 1 5B234BE3
 P 5900 3350
-F 0 "R21" V 5980 3350 50  0000 C CNN
+F 0 "R19" V 5980 3350 50  0000 C CNN
 F 1 "R" V 5900 3350 50  0000 C CNN
 F 2 "alex-library:R_Axial_Long6.3mm_Dia2.5mm_Pas15.24mm_Horizontal" V 5830 3350 50  0001 C CNN
@@
 $EndComp
 $Comp
-L R R22
+L R R20
 U 1 1 5B234BE4
 P 6150 3450
-F 0 "R22" V 6230 3450 50  0000 C CNN
+F 0 "R20" V 6230 3450 50  0000 C CNN
 F 1 "R" V 6150 3450 50  0000 C CNN
 F 2 "alex-library:R_Axial_Long6.3mm_Dia2.5mm_Pas15.24mm_Horizontal" V 6080 3450 50  0001 C CNN
@@
 $EndComp
 $Comp
-L R R23
+L R R21
 U 1 1 5B234BE5
 P 6400 3550
-F 0 "R23" V 6480 3550 50  0000 C CNN
+F 0 "R21" V 6480 3550 50  0000 C CNN
 F 1 "R" V 6400 3550 50  0000 C CNN
 F 2 "alex-library:R_Axial_Long6.3mm_Dia2.5mm_Pas15.24mm_Horizontal" V 6330 3550 50  0001 C CNN
@@
 $EndComp
 $Comp
-L R R24
+L R R22
 U 1 1 5B234BE6
 P 6650 3650
-F 0 "R24" V 6730 3650 50  0000 C CNN
+F 0 "R22" V 6730 3650 50  0000 C CNN
 F 1 "R" V 6650 3650 50  0000 C CNN
 F 2 "alex-library:R_Axial_Long6.3mm_Dia2.5mm_Pas15.24mm_Horizontal" V 6580 3650 50  0001 C CNN
@@
 $EndComp
 $Comp
-L R R25
+L R R23
 U 1 1 5B234BE7
 P 6900 3750
-F 0 "R25" V 6980 3750 50  0000 C CNN
+F 0 "R23" V 6980 3750 50  0000 C CNN
 F 1 "R" V 6900 3750 50  0000 C CNN
 F 2 "alex-library:R_Axial_Long6.3mm_Dia2.5mm_Pas15.24mm_Horizontal" V 6830 3750 50  0001 C CNN
@@
 $EndComp
 $Comp
-L R R26
+L R R24
 U 1 1 5B234BE8
 P 7150 3850
-F 0 "R26" V 7230 3850 50  0000 C CNN
+F 0 "R24" V 7230 3850 50  0000 C CNN
 F 1 "R" V 7150 3850 50  0000 C CNN
 F 2 "alex-library:R_Axial_Long6.3mm_Dia2.5mm_Pas15.24mm_Horizontal" V 7080 3850 50  0001 C CNN
@@
 	5350 3850 7000 3850
 $Comp
-L R R27
+L R R25
 U 1 1 5B234BE9
 P 7400 3950
-F 0 "R27" V 7480 3950 50  0000 C CNN
+F 0 "R25" V 7480 3950 50  0000 C CNN
 F 1 "R" V 7400 3950 50  0000 C CNN
 F 2 "alex-library:R_Axial_Long6.3mm_Dia2.5mm_Pas15.24mm_Horizontal" V 7330 3950 50  0001 C CNN
