File: Cube/PCB/Block Row Anode 8.sch (KiCad schematic (older format))
At the start: 10 parts

Commit message: Update
Update
Parts:
- removed C?: 100nF, symbol C
- removed R? (x8): R, symbol R
- removed U?: SN74HC595, symbol SN74HC595
- added C9: 100nF, symbol C
- added R44, R45, R46, R47, R48, R49, R50, R51: R, symbol R
- added U7: SN74HC595, symbol SN74HC595
Connections:
- net +5V: now also C9.1, U7.16 (VCC)
- net GND: now also C9.2, U7.13 (~OE), U7.8 (GND)
- net RCLK: now also U7.12 (RCLK)
- net R_QA: now also R44.1
- net R_QB: now also R45.1
- net R_QC: now also R46.1
- net R_QD: now also R47.1
- net R_QE: now also R48.1
- net R_QF: now also R49.1
- net R_QG: now also R50.1
- net R_QH: now also R51.1
- net R_QH': now also U7.9 (QH')
- net SER: now also U7.14 (SER)
- net SRCLK: now also U7.11 (SRCLK)
- new net: R45.2, U7.1 (QB)
- new net: R44.2, U7.15 (QA)
- new net: R46.2, U7.2 (QC)
- new net: R47.2, U7.3 (QD)
- new net: R48.2, U7.4 (QE)
- new net: R49.2, U7.5 (QF)
- new net: R50.2, U7.6 (QG)
- new net: R51.2, U7.7 (QH)
- new net ~SRCLR: U7.10 (~SRCLR)
Other:
- note added: "Choisir valeur de R\n130 Ohm pour une led rouge (5-(1.8+0.6))/0.02\n90 Ohm pour une led bleu (5-(3+0.6))/0.02"
- note removed: "Choisir valeur de R\n(5-(1.8+0.6))/0.02\n130 Ohm pour une led rouge\n120 Ohm pour une led bleu"
Changed lines of the file:
@@
 LIBS:valves
 LIBS:alex-library
+LIBS:Cube-8x8x8-512_LEDS-cache
 EELAYER 25 0
 EELAYER END
 $Descr A4 11693 8268
 encoding utf-8
-Sheet 4 12
+Sheet 9 12
 Title ""
 Date ""
@@
 $EndDescr
 $Comp
-L SN74HC595 U?
-U 1 1 5B2235DE
+L SN74HC595 U7
+U 1 1 5B2373DE
 P 4900 3650
-AR Path="/5B22355E/5B2235D3/5B2235DE" Ref="U?"  Part="1"
-AR Path="/5B22355E/5B22654D/5B2235DE" Ref="U?"  Part="1"
-F 0 "U?" H 4700 4200 60  0000 C CNN
+F 0 "U7" H 4700 4200 60  0000 C CNN
 F 1 "SN74HC595" H 4900 3100 60  0000 C CNN
 F 2 "" H 5250 3550 60  0001 C CNN
@@
 $EndComp
 $Comp
-L C C?
-U 1 1 5B223645
+L C C9
+U 1 1 5B2373DF
 P 3750 3000
-AR Path="/5B22355E/5B2235D3/5B223645" Ref="C?"  Part="1"
-AR Path="/5B22355E/5B22654D/5B223645" Ref="C?"  Part="1"
-F 0 "C?" H 3775 3100 50  0000 L CNN
+F 0 "C9" H 3775 3100 50  0000 L CNN
 F 1 "100nF" H 3775 2900 50  0000 L CNN
 F 2 "" H 3788 2850 50  0001 C CNN
@@
 $EndComp
 $Comp
-L +5V #PWR?
-U 1 1 5B223671
+L +5V #PWR34
+U 1 1 5B2373E0
 P 3750 2700
-AR Path="/5B22355E/5B2235D3/5B223671" Ref="#PWR?"  Part="1"
-AR Path="/5B22355E/5B22654D/5B223671" Ref="#PWR?"  Part="1"
-F 0 "#PWR?" H 3750 2550 50  0001 C CNN
+F 0 "#PWR34" H 3750 2550 50  0001 C CNN
 F 1 "+5V" H 3750 2840 50  0000 C CNN
 F 2 "" H 3750 2700 50  0001 C CNN
@@
 $EndComp
 $Comp
-L GND #PWR?
-U 1 1 5B223689
+L GND #PWR35
+U 1 1 5B2373E1
 P 3750 3300
-AR Path="/5B22355E/5B2235D3/5B223689" Ref="#PWR?"  Part="1"
-AR Path="/5B22355E/5B22654D/5B223689" Ref="#PWR?"  Part="1"
-F 0 "#PWR?" H 3750 3050 50  0001 C CNN
+F 0 "#PWR35" H 3750 3050 50  0001 C CNN
 F 1 "GND" H 3750 3150 50  0000 C CNN
 F 2 "" H 3750 3300 50  0001 C CNN
@@
 $EndComp
 $Comp
-L GND #PWR?
-U 1 1 5B2236C5
+L GND #PWR37
+U 1 1 5B2373E2
 P 4300 3400
-AR Path="/5B22355E/5B2235D3/5B2236C5" Ref="#PWR?"  Part="1"
-AR Path="/5B22355E/5B22654D/5B2236C5" Ref="#PWR?"  Part="1"
-F 0 "#PWR?" H 4300 3150 50  0001 C CNN
+F 0 "#PWR37" H 4300 3150 50  0001 C CNN
 F 1 "GND" H 4300 3250 50  0000 C CNN
 F 2 "" H 4300 3400 50  0001 C CNN
@@
 $EndComp
 $Comp
-L +5V #PWR?
-U 1 1 5B223752
-P 4000 3600
-AR Path="/5B22355E/5B22654D/5B223752" Ref="#PWR?"  Part="1"
-AR Path="/5B22355E/5B2235D3/5B223752" Ref="#PWR?"  Part="1"
-F 0 "#PWR?" H 4000 3450 50  0001 C CNN
-F 1 "+5V" H 4000 3740 50  0000 C CNN
-F 2 "" H 4000 3600 50  0001 C CNN
-F 3 "" H 4000 3600 50  0001 C CNN
-	1    4000 3600
-	1    0    0    -1
-$EndComp
-$Comp
-L GND #PWR?
-U 1 1 5B2237AC
+L GND #PWR36
+U 1 1 5B2373E3
 P 4000 4000
-AR Path="/5B22355E/5B22654D/5B2237AC" Ref="#PWR?"  Part="1"
-AR Path="/5B22355E/5B2235D3/5B2237AC" Ref="#PWR?"  Part="1"
-F 0 "#PWR?" H 4000 3750 50  0001 C CNN
+F 0 "#PWR36" H 4000 3750 50  0001 C CNN
 F 1 "GND" H 4000 3850 50  0000 C CNN
 F 2 "" H 4000 4000 50  0001 C CNN
@@
 	1    0    0    -1
 $EndComp
-Text HLabel 3100 3750 0    60   Input ~ 0
+Text HLabel 2200 3750 0    60   Input ~ 0
 SRCLK
-Text HLabel 3100 3850 0    60   Input ~ 0
+Text HLabel 2200 3850 0    60   Input ~ 0
 RCLK
-Text HLabel 3100 4350 0    60   Input ~ 0
+Text HLabel 2150 4350 0    60   Input ~ 0
 SER
 Text HLabel 7700 3250 2    60   Output ~ 0
@@
 R_QH'
 $Comp
-L R R?
-U 1 1 5B2238E0
+L R R44
+U 1 1 5B2373E4
 P 5650 3250
-AR Path="/5B22355E/5B2235D3/5B2238E0" Ref="R?"  Part="1"
-AR Path="/5B22355E/5B22654D/5B2238E0" Ref="R?"  Part="1"
-F 0 "R?" V 5730 3250 50  0000 C CNN
+F 0 "R44" V 5730 3250 50  0000 C CNN
 F 1 "R" V 5650 3250 50  0000 C CNN
 F 2 "" V 5580 3250 50  0001 C CNN
@@
 $EndComp
 $Comp
-L R R?
-U 1 1 5B223906
+L R R45
+U 1 1 5B2373E5
 P 5900 3350
-AR Path="/5B22355E/5B2235D3/5B223906" Ref="R?"  Part="1"
-AR Path="/5B22355E/5B22654D/5B223906" Ref="R?"  Part="1"
-F 0 "R?" V 5980 3350 50  0000 C CNN
+F 0 "R45" V 5980 3350 50  0000 C CNN
 F 1 "R" V 5900 3350 50  0000 C CNN
 F 2 "" V 5830 3350 50  0001 C CNN
@@
 $EndComp
 $Comp
-L R R?
-U 1 1 5B223932
+L R R46
+U 1 1 5B2373E6
 P 6150 3450
-AR Path="/5B22355E/5B2235D3/5B223932" Ref="R?"  Part="1"
-AR Path="/5B22355E/5B22654D/5B223932" Ref="R?"  Part="1"
-F 0 "R?" V 6230 3450 50  0000 C CNN
+F 0 "R46" V 6230 3450 50  0000 C CNN
 F 1 "R" V 6150 3450 50  0000 C CNN
 F 2 "" V 6080 3450 50  0001 C CNN
@@
 $EndComp
 $Comp
-L R R?
-U 1 1 5B2239C6
+L R R47
+U 1 1 5B2373E7
 P 6400 3550
-AR Path="/5B22355E/5B2235D3/5B2239C6" Ref="R?"  Part="1"
-AR Path="/5B22355E/5B22654D/5B2239C6" Ref="R?"  Part="1"
-F 0 "R?" V 6480 3550 50  0000 C CNN
+F 0 "R47" V 6480 3550 50  0000 C CNN
 F 1 "R" V 6400 3550 50  0000 C CNN
 F 2 "" V 6330 3550 50  0001 C CNN
@@
 $EndComp
 $Comp
-L R R?
-U 1 1 5B2239FA
+L R R48
+U 1 1 5B2373E8
 P 6650 3650
-AR Path="/5B22355E/5B2235D3/5B2239FA" Ref="R?"  Part="1"
-AR Path="/5B22355E/5B22654D/5B2239FA" Ref="R?"  Part="1"
-F 0 "R?" V 6730 3650 50  0000 C CNN
+F 0 "R48" V 6730 3650 50  0000 C CNN
 F 1 "R" V 6650 3650 50  0000 C CNN
 F 2 "" V 6580 3650 50  0001 C CNN
@@
 $EndComp
 $Comp
-L R R?
-U 1 1 5B223A31
+L R R49
+U 1 1 5B2373E9
 P 6900 3750
-AR Path="/5B22355E/5B2235D3/5B223A31" Ref="R?"  Part="1"
-AR Path="/5B22355E/5B22654D/5B223A31" Ref="R?"  Part="1"
-F 0 "R?" V 6980 3750 50  0000 C CNN
+F 0 "R49" V 6980 3750 50  0000 C CNN
 F 1 "R" V 6900 3750 50  0000 C CNN
 F 2 "" V 6830 3750 50  0001 C CNN
@@
 $EndComp
 $Comp
-L R R?
-U 1 1 5B223B39
+L R R50
+U 1 1 5B2373EA
 P 7150 3850
-AR Path="/5B22355E/5B2235D3/5B223B39" Ref="R?"  Part="1"
-AR Path="/5B22355E/5B22654D/5B223B39" Ref="R?"  Part="1"
-F 0 "R?" V 7230 3850 50  0000 C CNN
+F 0 "R50" V 7230 3850 50  0000 C CNN
 F 1 "R" V 7150 3850 50  0000 C CNN
 F 2 "" V 7080 3850 50  0001 C CNN
@@
 Connection ~ 3750 2800
 Wire Wire Line
-	4000 3600 4000 3650
-Wire Wire Line
-	4000 3650 4450 3650
-Wire Wire Line
 	4450 3950 4000 3950
 Wire Wire Line
@@
 	5350 3850 7000 3850
 $Comp
-L R R?
-U 1 1 5B2240C8
+L R R51
+U 1 1 5B2373EB
 P 7400 3950
-AR Path="/5B22355E/5B22654D/5B2240C8" Ref="R?"  Part="1"
-AR Path="/5B22355E/5B2235D3/5B2240C8" Ref="R?"  Part="1"
-F 0 "R?" V 7480 3950 50  0000 C CNN
+F 0 "R51" V 7480 3950 50  0000 C CNN
 F 1 "R" V 7400 3950 50  0000 C CNN
 F 2 "" V 7330 3950 50  0001 C CNN
@@
 Wire Wire Line
 	7550 3950 7700 3950
-Wire Wire Line
-	3100 3750 4450 3750
-Wire Wire Line
-	3100 3850 4450 3850
-Wire Wire Line
-	4450 4050 4250 4050
-Wire Wire Line
-	4250 4050 4250 4350
-Wire Wire Line
-	4250 4350 3100 4350
-Text Notes 6850 2900 2    60   ~ 0
-Choisir valeur de R\n(5-(1.8+0.6))/0.02\n130 Ohm pour une led rouge\n120 Ohm pour une led bleu
+Text Notes 8150 2950 2    60   ~ 0
+Choisir valeur de R\n130 Ohm pour une led rouge (5-(1.8+0.6))/0.02\n90 Ohm pour une led bleu (5-(3+0.6))/0.02
+Wire Wire Line
+	2200 3750 4450 3750
+Wire Wire Line
+	2200 3850 4450 3850
+Wire Wire Line
+	2150 4350 4300 4350
+Wire Wire Line
+	4300 4350 4300 4050
+Wire Wire Line
+	4300 4050 4450 4050
+Text HLabel 2200 3550 0    60   Input ~ 0
+~SRCLR
+Wire Wire Line
+	2200 3550 3000 3550
+Wire Wire Line
+	3000 3550 3000 3650
+Wire Wire Line
+	3000 3650 4450 3650
 $EndSCHEMATC

Commit message: Update project
Remove a image corrupted -_-
Parts:
- C9: footprint (none) -> alex-library:C-P_5.08-L_7.5-H_6-P_2.5
- R44, R45, R46, R47, R48, R49, R50, R51: footprint (none) -> alex-library:R_Axial_Long6.3mm_Dia2.5mm_Pas15.24mm_Horizontal
- U7: footprint (none) -> alex-library:DIP-16_W7.62mm_LongPads
Changed lines of the file:
@@
 F 0 "U7" H 4700 4200 60  0000 C CNN
 F 1 "SN74HC595" H 4900 3100 60  0000 C CNN
-F 2 "" H 5250 3550 60  0001 C CNN
+F 2 "alex-library:DIP-16_W7.62mm_LongPads" H 5250 3550 60  0001 C CNN
 F 3 "" H 5250 3550 60  0001 C CNN
 	1    4900 3650
@@
 F 0 "C9" H 3775 3100 50  0000 L CNN
 F 1 "100nF" H 3775 2900 50  0000 L CNN
-F 2 "" H 3788 2850 50  0001 C CNN
+F 2 "alex-library:C-P_5.08-L_7.5-H_6-P_2.5" H 3788 2850 50  0001 C CNN
 F 3 "" H 3750 3000 50  0001 C CNN
 	1    3750 3000
@@
 $EndComp
 $Comp
-L +5V #PWR34
+L +5V #PWR042
 U 1 1 5B2373E0
 P 3750 2700
-F 0 "#PWR34" H 3750 2550 50  0001 C CNN
+F 0 "#PWR042" H 3750 2550 50  0001 C CNN
 F 1 "+5V" H 3750 2840 50  0000 C CNN
 F 2 "" H 3750 2700 50  0001 C CNN
@@
 $EndComp
 $Comp
-L GND #PWR35
+L GND #PWR043
 U 1 1 5B2373E1
 P 3750 3300
-F 0 "#PWR35" H 3750 3050 50  0001 C CNN
+F 0 "#PWR043" H 3750 3050 50  0001 C CNN
 F 1 "GND" H 3750 3150 50  0000 C CNN
 F 2 "" H 3750 3300 50  0001 C CNN
@@
 $EndComp
 $Comp
-L GND #PWR37
+L GND #PWR044
 U 1 1 5B2373E2
 P 4300 3400
-F 0 "#PWR37" H 4300 3150 50  0001 C CNN
+F 0 "#PWR044" H 4300 3150 50  0001 C CNN
 F 1 "GND" H 4300 3250 50  0000 C CNN
 F 2 "" H 4300 3400 50  0001 C CNN
@@
 $EndComp
 $Comp
-L GND #PWR36
+L GND #PWR045
 U 1 1 5B2373E3
 P 4000 4000
-F 0 "#PWR36" H 4000 3750 50  0001 C CNN
+F 0 "#PWR045" H 4000 3750 50  0001 C CNN
 F 1 "GND" H 4000 3850 50  0000 C CNN
 F 2 "" H 4000 4000 50  0001 C CNN
@@
 F 0 "R44" V 5730 3250 50  0000 C CNN
 F 1 "R" V 5650 3250 50  0000 C CNN
-F 2 "" V 5580 3250 50  0001 C CNN
+F 2 "alex-library:R_Axial_Long6.3mm_Dia2.5mm_Pas15.24mm_Horizontal" V 5580 3250 50  0001 C CNN
 F 3 "" H 5650 3250 50  0001 C CNN
 	1    5650 3250
@@
 F 0 "R45" V 5980 3350 50  0000 C CNN
 F 1 "R" V 5900 3350 50  0000 C CNN
-F 2 "" V 5830 3350 50  0001 C CNN
+F 2 "alex-library:R_Axial_Long6.3mm_Dia2.5mm_Pas15.24mm_Horizontal" V 5830 3350 50  0001 C CNN
 F 3 "" H 5900 3350 50  0001 C CNN
 	1    5900 3350
@@
 F 0 "R46" V 6230 3450 50  0000 C CNN
 F 1 "R" V 6150 3450 50  0000 C CNN
-F 2 "" V 6080 3450 50  0001 C CNN
+F 2 "alex-library:R_Axial_Long6.3mm_Dia2.5mm_Pas15.24mm_Horizontal" V 6080 3450 50  0001 C CNN
 F 3 "" H 6150 3450 50  0001 C CNN
 	1    6150 3450
@@
 F 0 "R47" V 6480 3550 50  0000 C CNN
 F 1 "R" V 6400 3550 50  0000 C CNN
-F 2 "" V 6330 3550 50  0001 C CNN
+F 2 "alex-library:R_Axial_Long6.3mm_Dia2.5mm_Pas15.24mm_Horizontal" V 6330 3550 50  0001 C CNN
 F 3 "" H 6400 3550 50  0001 C CNN
 	1    6400 3550
@@
 F 0 "R48" V 6730 3650 50  0000 C CNN
 F 1 "R" V 6650 3650 50  0000 C CNN
-F 2 "" V 6580 3650 50  0001 C CNN
+F 2 "alex-library:R_Axial_Long6.3mm_Dia2.5mm_Pas15.24mm_Horizontal" V 6580 3650 50  0001 C CNN
 F 3 "" H 6650 3650 50  0001 C CNN
 	1    6650 3650
@@
 F 0 "R49" V 6980 3750 50  0000 C CNN
 F 1 "R" V 6900 3750 50  0000 C CNN
-F 2 "" V 6830 3750 50  0001 C CNN
+F 2 "alex-library:R_Axial_Long6.3mm_Dia2.5mm_Pas15.24mm_Horizontal" V 6830 3750 50  0001 C CNN
 F 3 "" H 6900 3750 50  0001 C CNN
 	1    6900 3750
@@
 F 0 "R50" V 7230 3850 50  0000 C CNN
 F 1 "R" V 7150 3850 50  0000 C CNN
-F 2 "" V 7080 3850 50  0001 C CNN
+F 2 "alex-library:R_Axial_Long6.3mm_Dia2.5mm_Pas15.24mm_Horizontal" V 7080 3850 50  0001 C CNN
 F 3 "" H 7150 3850 50  0001 C CNN
 	1    7150 3850
@@
 F 0 "R51" V 7480 3950 50  0000 C CNN
 F 1 "R" V 7400 3950 50  0000 C CNN
-F 2 "" V 7330 3950 50  0001 C CNN
+F 2 "alex-library:R_Axial_Long6.3mm_Dia2.5mm_Pas15.24mm_Horizontal" V 7330 3950 50  0001 C CNN
 F 3 "" H 7400 3950 50  0001 C CNN
 	1    7400 3950

Commit message: Update
Update
Add New restistor in Base Q1, Q2, Q3, Q4, Q5, Q6, Q7, Q8
New version PCB
New rename components
Parts:
- renumbered R44 to R42, R45 to R43, R46 to R44, R47 to R45, R48 to R46, R49 to R47, R50 to R48, R51 to R49
Changed lines of the file:
@@
 R_QH'
 $Comp
-L R R44
+L R R42
 U 1 1 5B2373E4
 P 5650 3250
-F 0 "R44" V 5730 3250 50  0000 C CNN
+F 0 "R42" V 5730 3250 50  0000 C CNN
 F 1 "R" V 5650 3250 50  0000 C CNN
 F 2 "alex-library:R_Axial_Long6.3mm_Dia2.5mm_Pas15.24mm_Horizontal" V 5580 3250 50  0001 C CNN
@@
 $EndComp
 $Comp
-L R R45
+L R R43
 U 1 1 5B2373E5
 P 5900 3350
-F 0 "R45" V 5980 3350 50  0000 C CNN
+F 0 "R43" V 5980 3350 50  0000 C CNN
 F 1 "R" V 5900 3350 50  0000 C CNN
 F 2 "alex-library:R_Axial_Long6.3mm_Dia2.5mm_Pas15.24mm_Horizontal" V 5830 3350 50  0001 C CNN
@@
 $EndComp
 $Comp
-L R R46
+L R R44
 U 1 1 5B2373E6
 P 6150 3450
-F 0 "R46" V 6230 3450 50  0000 C CNN
+F 0 "R44" V 6230 3450 50  0000 C CNN
 F 1 "R" V 6150 3450 50  0000 C CNN
 F 2 "alex-library:R_Axial_Long6.3mm_Dia2.5mm_Pas15.24mm_Horizontal" V 6080 3450 50  0001 C CNN
@@
 $EndComp
 $Comp
-L R R47
+L R R45
 U 1 1 5B2373E7
 P 6400 3550
-F 0 "R47" V 6480 3550 50  0000 C CNN
+F 0 "R45" V 6480 3550 50  0000 C CNN
 F 1 "R" V 6400 3550 50  0000 C CNN
 F 2 "alex-library:R_Axial_Long6.3mm_Dia2.5mm_Pas15.24mm_Horizontal" V 6330 3550 50  0001 C CNN
@@
 $EndComp
 $Comp
-L R R48
+L R R46
 U 1 1 5B2373E8
 P 6650 3650
-F 0 "R48" V 6730 3650 50  0000 C CNN
+F 0 "R46" V 6730 3650 50  0000 C CNN
 F 1 "R" V 6650 3650 50  0000 C CNN
 F 2 "alex-library:R_Axial_Long6.3mm_Dia2.5mm_Pas15.24mm_Horizontal" V 6580 3650 50  0001 C CNN
@@
 $EndComp
 $Comp
-L R R49
+L R R47
 U 1 1 5B2373E9
 P 6900 3750
-F 0 "R49" V 6980 3750 50  0000 C CNN
+F 0 "R47" V 6980 3750 50  0000 C CNN
 F 1 "R" V 6900 3750 50  0000 C CNN
 F 2 "alex-library:R_Axial_Long6.3mm_Dia2.5mm_Pas15.24mm_Horizontal" V 6830 3750 50  0001 C CNN
@@
 $EndComp
 $Comp
-L R R50
+L R R48
 U 1 1 5B2373EA
 P 7150 3850
-F 0 "R50" V 7230 3850 50  0000 C CNN
+F 0 "R48" V 7230 3850 50  0000 C CNN
 F 1 "R" V 7150 3850 50  0000 C CNN
 F 2 "alex-library:R_Axial_Long6.3mm_Dia2.5mm_Pas15.24mm_Horizontal" V 7080 3850 50  0001 C CNN
@@
 	5350 3850 7000 3850
 $Comp
-L R R51
+L R R49
 U 1 1 5B2373EB
 P 7400 3950
-F 0 "R51" V 7480 3950 50  0000 C CNN
+F 0 "R49" V 7480 3950 50  0000 C CNN
 F 1 "R" V 7400 3950 50  0000 C CNN
 F 2 "alex-library:R_Axial_Long6.3mm_Dia2.5mm_Pas15.24mm_Horizontal" V 7330 3950 50  0001 C CNN
