File: Cube/PCB/Cube-8x8x8-512_LEDS.kicad_pcb (KiCad board)
At the start: 2 copper layers, 200 x 200 mm, 154 parts, among them J1 Conn_01x02_Male, J10 Conn_01x10_Male, J11 Conn_01x10_Male, J12 Conn_01x10_Male, J13 Conn_01x04_Male, J14 Conn_01x08_Male, J2 Conn_01x09_Male, J3 Conn_01x04_Male, J4 Conn_01x10_Male, J5 Conn_01x06_Male, J6 Conn_01x06_Male, J7 Conn_01x10_Male, J8 Conn_01x10_Male, J9 Conn_01x10_Male, Q1 PN2222A, Q2 PN2222A, Q3 PN2222A, Q4 PN2222A, Q5 PN2222A, Q6 PN2222A, Q7 PN2222A, Q8 PN2222A, SW1 Chevron, SW10 Chevron, SW11 Chevron, SW12 Chevron, SW13 Chevron, SW14 Chevron, SW15 Chevron, SW16 Chevron, SW17 Chevron, SW18 Chevron, SW19 Chevron, SW2 Chevron, SW20 Chevron, SW21 Chevron, SW22 Chevron, SW23 Chevron, SW24 Chevron, SW25 Chevron, SW26 Chevron, SW27 Chevron, SW28 Chevron, SW29 Chevron, SW3 Chevron, SW30 Chevron, SW31 Chevron, SW32 Chevron, SW33 Chevron, SW34 Chevron, SW36 Chevron, SW37 Chevron, SW38 Chevron, SW39 Chevron, SW4 Chevron, SW5 Chevron, SW6 Chevron, SW7 Chevron, SW8 Chevron, SW9 Chevron, U1 LM317_A, U10 SN74HC595, U2 SN74HC595, U3 SN74HC595, U4 SN74HC595, U5 SN74HC595, U6 SN74HC595, U7 SN74HC595, U8 SN74HC595, U9 SN74HC595

Commit message: Update
Update
Parts:
- added SW35: Chevron, alex-library:Chevron-E1, B.Cu at (176.5, 80.0)
- SW10, SW11, SW12, SW13, SW14, SW15, SW16, SW17, SW18, SW19, SW20, SW21, SW22, SW23, SW24, SW25, SW26, SW27, SW28, SW29, SW3, SW30, SW31, SW32, SW33, SW34, SW36, SW37, SW38, SW4, SW5, SW6, SW7, SW8, SW9: moved to B.Cu
- moved SW38 212.9 mm to (176.5, 83.8), turned to 180 degrees
- moved SW36 208.5 mm to (176.5, 76.2), turned to 180 degrees
- moved SW34 197.3 mm to (171.4, 110.5), turned to 180 degrees
- moved SW37 196.6 mm to (176.5, 72.4), turned to 180 degrees
- moved SW33 193.3 mm to (171.4, 99.1), turned to 180 degrees
- moved SW24 193.1 mm to (171.4, 141.0), turned to 180 degrees
- moved SW18 190.4 mm to (171.4, 186.7), turned to 180 degrees
- moved SW32 185.7 mm to (171.4, 102.9), turned to 180 degrees
- moved SW8 184.0 mm to (171.4, 217.2), turned to 180 degrees
- moved SW31 180.8 mm to (171.4, 106.7), turned to 180 degrees
- moved SW16 178.5 mm to (171.4, 179.1), turned to 180 degrees
- moved SW26 175.4 mm to (171.4, 148.6), turned to 180 degrees
- moved SW7 174.7 mm to (171.4, 221.0), turned to 180 degrees
- moved SW10 173.6 mm to (171.4, 224.8), turned to 180 degrees
- moved SW15 169.2 mm to (171.4, 182.9), turned to 180 degrees
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Routing:
- net /Matrice/A8: track 0.00 -> 154.8 mm
- net /Matrice/A7: track 0.00 -> 151.0 mm
- net /Matrice/A6: track 0.00 -> 147.2 mm
- net /Matrice/A5: track 0.00 -> 143.4 mm
- net /Matrice/A1: track 0.00 -> 135.3 mm
- net /Matrice/A2: track 0.00 -> 127.2 mm
- net /Matrice/A3: track 0.00 -> 119.0 mm
- net /Matrice/A4: track 0.00 -> 109.8 mm
- net /Matrice/A39: track 183.6 -> 129.2 mm
- net /Matrice/A37: track 173.9 -> 119.5 mm
- net /Matrice/A40: track 188.4 -> 134.1 mm
- net /Matrice/A38: track 178.7 -> 124.3 mm
- net /Matrice/A55: track 184.9 -> 133.4 mm
- net /Matrice/A54: track 180.0 -> 128.5 mm
- net /Matrice/A53: track 175.1 -> 123.7 mm
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- added copper zone on B.Cu, net GND
Other:
- board size 200 x 200 mm -> 180 x 195 mm

Commit message: Update
Update
Parts:
- SW1, SW2, SW39: moved to B.Cu
- moved SW1 173.5 mm to (236.2, 241.3)
- moved SW2 156.5 mm to (236.2, 237.5)
- moved SW39 144.1 mm to (257.8, 245.1), turned to 270 degrees
- moved J6 131.4 mm to (260.4, 251.5)
- moved J1 128.8 mm to (240.0, 64.8)
- moved J5 128.7 mm to (200.7, 99.1), turned to 90 degrees
- moved J2 126.3 mm to (221.0, 64.8), turned to 180 degrees
- moved R1 126.1 mm to (257.8, 237.5), turned to 180 degrees
- moved C3 114.0 mm to (237.5, 87.6), turned to 90 degrees
- moved C1 113.5 mm to (221.0, 87.6), turned to 90 degrees
- moved C2 109.2 mm to (233.7, 87.6), turned to 90 degrees
- moved D3 105.0 mm to (224.8, 99.1)
- moved RV1 102.6 mm to (252.7, 87.6), turned to 270 degrees
- moved J4 102.3 mm to (218.4, 111.8)
- moved U1 95.5 mm to (240.0, 92.7), turned to 180 degrees
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Routing:
- net +5V: track 57.1 -> 703.7 mm, vias 0 -> 11
- net RCLK: track 6.88 -> 472.9 mm, vias 0 -> 10
- net SRCLK: track 6.35 -> 426.8 mm, vias 0 -> 10
- net ~SRCLR: track 6.88 -> 402.1 mm, vias 0 -> 10
- net /Matrice/BlockLayersCatodes/R_QH': track 0.00 -> 285.3 mm, vias 0 -> 1
- net SRCLR_CMD: track 0.00 -> 212.4 mm
- net RCLK_CMD: track 0.00 -> 168.5 mm, vias 0 -> 3
- net SRCLK_CMD: track 0.00 -> 168.0 mm, vias 0 -> 3
- net SER_8: track 0.00 -> 156.0 mm, vias 0 -> 2
- net SER_3: track 0.00 -> 149.9 mm, vias 0 -> 2
- net SER_5: track 0.00 -> 145.8 mm, vias 0 -> 2
- net SER_START: track 0.00 -> 134.2 mm, vias 0 -> 1
- net SER_7: track 0.00 -> 132.1 mm, vias 0 -> 2
- net SER_6: track 0.00 -> 113.1 mm, vias 0 -> 2
- net Net-(J2-Pad2): track 0.00 -> 107.8 mm, vias 0 -> 1
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- added copper zone on F.Cu, net GND

Commit message: Update Project
Update Project
Other:
- rule trace_min: 0.2 -> 0.3
Changed lines of the file:
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@@
   )
   (setup
-    (last_trace_width 0.8)
+    (last_trace_width 0.25)
     (user_trace_width 0.6)
     (user_trace_width 0.8)
@@
     (zone_clearance 0.508)
     (zone_45_only no)
-    (trace_min 0.2)
+    (trace_min 0.3)
     (segment_width 0.2)
     (edge_width 0.1)
@@
     (visible_elements 7FFFFFFF)
     (pcbplotparams
-      (layerselection 0x00030_80000001)
+      (layerselection 0x01000_80000001)
       (usegerberextensions false)
       (excludeedgelayer true)
@@
       (drillshape 0)
       (scaleselection 1)
-      (outputdirectory ""))
+      (outputdirectory Logique-Commande-Cube-8x8x8-512-Leds-Gerber/))
   )
   (net 0 "")
@@
   (segment (start 210.82 93.853) (end 210.693 93.98) (width 0.8) (layer F.Cu) (net 27))
   (segment (start 257.81 251.46) (end 257.81 247.65) (width 0.8) (layer B.Cu) (net 28))
-  (segment (start 237.744 119.38) (end 237.744 125.984) (width 0.8) (layer F.Cu) (net 29) (status 400000))
+  (segment (start 237.744 119.38) (end 237.744 125.984) (width 0.8) (layer F.Cu) (net 29))
   (segment (start 266.7 128.27) (end 266.7 223.52) (width 0.8) (layer F.Cu) (net 29))
   (segment (start 265.43 127) (end 266.7 128.27) (width 0.8) (layer F.Cu) (net 29))
@@
   (via (at 261.62 223.52) (size 1.4) (drill 0.8) (layers F.Cu B.Cu) (net 29))
   (segment (start 260.35 238.76) (end 260.35 251.46) (width 0.8) (layer B.Cu) (net 29))
-  (segment (start 245.364 119.38) (end 245.364 123.444) (width 0.8) (layer F.Cu) (net 30) (status 400000))
+  (segment (start 245.364 119.38) (end 245.364 123.444) (width 0.8) (layer F.Cu) (net 30))
   (via (at 269.24 219.71) (size 1.4) (drill 0.8) (layers F.Cu B.Cu) (net 30))
   (segment (start 269.24 219.71) (end 271.78 217.17) (width 0.8) (layer F.Cu) (net 30))
@@
   (segment (start 252.73 219.71) (end 250.19 219.71) (width 0.8) (layer B.Cu) (net 180))
   (segment (start 262.89 193.04) (end 254.635 193.04) (width 0.8) (layer B.Cu) (net 180))
-  (segment (start 240.284 119.38) (end 240.284 124.714) (width 0.8) (layer F.Cu) (net 181) (status 400000))
+  (segment (start 240.284 119.38) (end 240.284 124.714) (width 0.8) (layer F.Cu) (net 181))
   (segment (start 241.3 125.73) (end 266.7 125.73) (width 0.8) (layer F.Cu) (net 181))
   (segment (start 266.7 125.73) (end 267.97 127) (width 0.8) (layer F.Cu) (net 181))

Commit message: Update
Update
Add New restistor in Base Q1, Q2, Q3, Q4, Q5, Q6, Q7, Q8
New version PCB
New rename components
Parts:
- removed D3: 1N4007, alex-library:D_DO-41_Pas12.70mm_Horizontal
- removed RV1: 470, alex-library:Potentiometer_Trimmer_Bourns_3296X
- added R68: 1,1K, alex-library:R_Axial_Long6.3mm_Dia2.5mm_Pas15.24mm_Horizontal, F.Cu at (165.1, 66.0)
- added R69: 1,1K, alex-library:R_Axial_Long6.3mm_Dia2.5mm_Pas15.24mm_Horizontal, F.Cu at (165.1, 69.8)
- added R70: 1,1K, alex-library:R_Axial_Long6.3mm_Dia2.5mm_Pas15.24mm_Horizontal, F.Cu at (165.1, 73.7)
- added R71: 1,1K, alex-library:R_Axial_Long6.3mm_Dia2.5mm_Pas15.24mm_Horizontal, F.Cu at (165.1, 77.5)
- added R72: 1,1K, alex-library:R_Axial_Long6.3mm_Dia2.5mm_Pas15.24mm_Horizontal, F.Cu at (165.1, 81.3)
- added R73: 1,1K, alex-library:R_Axial_Long6.3mm_Dia2.5mm_Pas15.24mm_Horizontal, F.Cu at (165.1, 85.1)
- R2: value 240 -> R
- R3: value 390 -> R
- R66, R67: value R -> 1,1K
- U1: value LM317_A -> L7805
- moved R66 152.8 mm to (165.1, 57.1), turned to 180 degrees
- moved R67 147.3 mm to (165.1, 62.2), turned to 180 degrees
- moved R3 130.7 mm to (194.3, 214.6), turned to 0 degrees
- moved R11 117.7 mm to (114.3, 174.0), turned to 0 degrees
- moved R2 117.2 mm to (194.3, 210.8)
- moved R43 116.9 mm to (114.3, 97.8), turned to 0 degrees
- moved R10 115.3 mm to (114.3, 170.2), turned to 0 degrees
- moved R59 115.2 mm to (114.3, 212.1), turned to 0 degrees
- moved R42 114.5 mm to (114.3, 94.0), turned to 0 degrees
- moved R27 113.8 mm to (114.3, 135.9), turned to 0 degrees
- moved R26 110.9 mm to (114.3, 132.1), turned to 0 degrees
- moved R58 110.6 mm to (114.3, 208.3), turned to 0 degrees
- moved R51 105.6 mm to (194.3, 188.0), turned to 0 degrees
- moved R50 104.1 mm to (194.3, 184.2), turned to 0 degrees
- moved R18 53.6 mm to (194.3, 157.5), turned to 0 degrees
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Connections:
- D2 pad 1: Net-(C3-Pad1) -> +5V
- D2 pad 2: Net-(D2-Pad2) -> Net-(C3-Pad1)
- R10 pad 1: /Matrice/A7 -> /Matrice/A25
- R11 pad 1: /Matrice/A8 -> /Matrice/A26
- R12 pad 1: /Matrice/A25 -> /Matrice/A27
- R13 pad 1: /Matrice/A26 -> /Matrice/A28
- R14 pad 1: /Matrice/A27 -> /Matrice/A29
- R15 pad 1: /Matrice/A28 -> /Matrice/A30
- R16 pad 1: /Matrice/A29 -> /Matrice/A31
- R17 pad 1: /Matrice/A30 -> /Matrice/A32
- R18 pad 1: /Matrice/A31 -> /Matrice/A33
- R19 pad 1: /Matrice/A32 -> /Matrice/A34
- R2 pad 1: Net-(C3-Pad1) -> /Matrice/A1
- R20 pad 1: /Matrice/A33 -> /Matrice/A35
- R21 pad 1: /Matrice/A34 -> /Matrice/A36
- R22 pad 1: /Matrice/A35 -> /Matrice/A37
- R23 pad 1: /Matrice/A36 -> /Matrice/A38
- R24 pad 1: /Matrice/A37 -> /Matrice/A39
- R25 pad 1: /Matrice/A38 -> /Matrice/A40
- R26 pad 1: /Matrice/A39 -> /Matrice/A41
- R27 pad 1: /Matrice/A40 -> /Matrice/A42
- R28 pad 1: /Matrice/A41 -> /Matrice/A43
- R29 pad 1: /Matrice/A42 -> /Matrice/A44
- R3 pad 1: Net-(R2-Pad2) -> /Matrice/A2
- R3 pad 2: Net-(D2-Pad2) -> Net-(R3-Pad2)
- R30 pad 1: /Matrice/A43 -> /Matrice/A45
- R31 pad 1: /Matrice/A44 -> /Matrice/A46
- R32 pad 1: /Matrice/A45 -> /Matrice/A47
- R33 pad 1: /Matrice/A46 -> /Matrice/A48
- R34 pad 1: /Matrice/A47 -> /Matrice/A49
- R35 pad 1: /Matrice/A48 -> /Matrice/A50
- R36 pad 1: /Matrice/A49 -> /Matrice/A51
- R37 pad 1: /Matrice/A50 -> /Matrice/A52
- R38 pad 1: /Matrice/A51 -> /Matrice/A53
- R39 pad 1: /Matrice/A52 -> /Matrice/A54
- R4 pad 1: /Matrice/A1 -> /Matrice/A3
- R40 pad 1: /Matrice/A53 -> /Matrice/A55
- R41 pad 1: /Matrice/A54 -> /Matrice/A56
- R42 pad 1: /Matrice/A55 -> /Matrice/A57
- R43 pad 1: /Matrice/A56 -> /Matrice/A58
- R44 pad 1: /Matrice/A57 -> /Matrice/A59
- R45 pad 1: /Matrice/A58 -> /Matrice/A60
- R46 pad 1: /Matrice/A59 -> /Matrice/A61
- R47 pad 1: /Matrice/A60 -> /Matrice/A62
- R48 pad 1: /Matrice/A61 -> /Matrice/A63
- R49 pad 1: /Matrice/A62 -> /Matrice/A64
- R5 pad 1: /Matrice/A2 -> /Matrice/A4
- R50 pad 1: /Matrice/A63 -> /Matrice/A17
- R51 pad 1: /Matrice/A64 -> /Matrice/A18
- R52 pad 1: /Matrice/A17 -> /Matrice/A19
- R53 pad 1: /Matrice/A18 -> /Matrice/A20
- R54 pad 1: /Matrice/A19 -> /Matrice/A21
- R55 pad 1: /Matrice/A20 -> /Matrice/A22
- R56 pad 1: /Matrice/A21 -> /Matrice/A23
- R57 pad 1: /Matrice/A22 -> /Matrice/A24
- R58 pad 1: /Matrice/A23 -> /Matrice/A9
- R59 pad 1: /Matrice/A24 -> /Matrice/A10
- R6 pad 1: /Matrice/A3 -> /Matrice/A5
- R60 pad 1: /Matrice/A9 -> /Matrice/A11
- R61 pad 1: /Matrice/A10 -> /Matrice/A12
- R62 pad 1: /Matrice/A11 -> /Matrice/A13
- R63 pad 1: /Matrice/A12 -> /Matrice/A14
- R64 pad 1: /Matrice/A13 -> /Matrice/A15
- R65 pad 1: /Matrice/A14 -> /Matrice/A16
- R66 pad 1: /Matrice/A15 -> Net-(R66-Pad1)
- R66 pad 2: Net-(R66-Pad2) -> Net-(Q1-Pad2)
- R67 pad 1: /Matrice/A16 -> Net-(R67-Pad1)
- R67 pad 2: Net-(R67-Pad2) -> Net-(Q2-Pad2)
- R7 pad 1: /Matrice/A4 -> /Matrice/A6
- R8 pad 1: /Matrice/A5 -> /Matrice/A7
- R9 pad 1: /Matrice/A6 -> /Matrice/A8
- U1 pad 1: Net-(D2-Pad2) -> Net-(C1-Pad1)
- U1 pad 2: Net-(C3-Pad1) -> GND
- U1 pad 3: Net-(C1-Pad1) -> Net-(C3-Pad1)
- U10 pad 1: Net-(Q2-Pad2) -> Net-(R67-Pad1)
- U10 pad 15: Net-(Q1-Pad2) -> Net-(R66-Pad1)
- U10 pad 2: Net-(Q3-Pad2) -> Net-(R68-Pad1)
- U10 pad 3: Net-(Q4-Pad2) -> Net-(R69-Pad1)
- U10 pad 4: Net-(Q5-Pad2) -> Net-(R70-Pad1)
- U10 pad 5: Net-(Q6-Pad2) -> Net-(R71-Pad1)
- U10 pad 6: Net-(Q7-Pad2) -> Net-(R72-Pad1)
- U10 pad 7: Net-(Q8-Pad2) -> Net-(R73-Pad1)
- U2 pad 1: Net-(R5-Pad2) -> Net-(R3-Pad2)
- U2 pad 15: Net-(R4-Pad2) -> Net-(R2-Pad2)
- U2 pad 2: Net-(R6-Pad2) -> Net-(R4-Pad2)
- U2 pad 3: Net-(R7-Pad2) -> Net-(R5-Pad2)
- U2 pad 4: Net-(R8-Pad2) -> Net-(R6-Pad2)
- U2 pad 5: Net-(R9-Pad2) -> Net-(R7-Pad2)
- U2 pad 6: Net-(R10-Pad2) -> Net-(R8-Pad2)
- U2 pad 7: Net-(R11-Pad2) -> Net-(R9-Pad2)
- U3 pad 1: Net-(R13-Pad2) -> Net-(R11-Pad2)
- U3 pad 15: Net-(R12-Pad2) -> Net-(R10-Pad2)
- U3 pad 2: Net-(R14-Pad2) -> Net-(R12-Pad2)
- U3 pad 3: Net-(R15-Pad2) -> Net-(R13-Pad2)
- U3 pad 4: Net-(R16-Pad2) -> Net-(R14-Pad2)
- U3 pad 5: Net-(R17-Pad2) -> Net-(R15-Pad2)
- U3 pad 6: Net-(R18-Pad2) -> Net-(R16-Pad2)
- U3 pad 7: Net-(R19-Pad2) -> Net-(R17-Pad2)
- U4 pad 1: Net-(R21-Pad2) -> Net-(R19-Pad2)
- U4 pad 15: Net-(R20-Pad2) -> Net-(R18-Pad2)
- U4 pad 2: Net-(R22-Pad2) -> Net-(R20-Pad2)
- U4 pad 3: Net-(R23-Pad2) -> Net-(R21-Pad2)
- U4 pad 4: Net-(R24-Pad2) -> Net-(R22-Pad2)
- U4 pad 5: Net-(R25-Pad2) -> Net-(R23-Pad2)
- U4 pad 6: Net-(R26-Pad2) -> Net-(R24-Pad2)
- U4 pad 7: Net-(R27-Pad2) -> Net-(R25-Pad2)
- U5 pad 1: Net-(R29-Pad2) -> Net-(R27-Pad2)
- U5 pad 15: Net-(R28-Pad2) -> Net-(R26-Pad2)
- U5 pad 2: Net-(R30-Pad2) -> Net-(R28-Pad2)
- U5 pad 3: Net-(R31-Pad2) -> Net-(R29-Pad2)
- U5 pad 4: Net-(R32-Pad2) -> Net-(R30-Pad2)
- U5 pad 5: Net-(R33-Pad2) -> Net-(R31-Pad2)
- U5 pad 6: Net-(R34-Pad2) -> Net-(R32-Pad2)
- U5 pad 7: Net-(R35-Pad2) -> Net-(R33-Pad2)
- U6 pad 1: Net-(R37-Pad2) -> Net-(R35-Pad2)
- U6 pad 15: Net-(R36-Pad2) -> Net-(R34-Pad2)
- U6 pad 2: Net-(R38-Pad2) -> Net-(R36-Pad2)
- U6 pad 3: Net-(R39-Pad2) -> Net-(R37-Pad2)
- U6 pad 4: Net-(R40-Pad2) -> Net-(R38-Pad2)
- U6 pad 5: Net-(R41-Pad2) -> Net-(R39-Pad2)
- U6 pad 6: Net-(R42-Pad2) -> Net-(R40-Pad2)
- U6 pad 7: Net-(R43-Pad2) -> Net-(R41-Pad2)
- U7 pad 1: Net-(R45-Pad2) -> Net-(R43-Pad2)
- U7 pad 15: Net-(R44-Pad2) -> Net-(R42-Pad2)
- U7 pad 2: Net-(R46-Pad2) -> Net-(R44-Pad2)
- U7 pad 3: Net-(R47-Pad2) -> Net-(R45-Pad2)
- U7 pad 4: Net-(R48-Pad2) -> Net-(R46-Pad2)
- U7 pad 5: Net-(R49-Pad2) -> Net-(R47-Pad2)
- U7 pad 6: Net-(R50-Pad2) -> Net-(R48-Pad2)
- U7 pad 7: Net-(R51-Pad2) -> Net-(R49-Pad2)
- U8 pad 1: Net-(R53-Pad2) -> Net-(R51-Pad2)
- U8 pad 15: Net-(R52-Pad2) -> Net-(R50-Pad2)
- U8 pad 2: Net-(R54-Pad2) -> Net-(R52-Pad2)
- U8 pad 3: Net-(R55-Pad2) -> Net-(R53-Pad2)
- U8 pad 4: Net-(R56-Pad2) -> Net-(R54-Pad2)
- U8 pad 5: Net-(R57-Pad2) -> Net-(R55-Pad2)
- U8 pad 6: Net-(R58-Pad2) -> Net-(R56-Pad2)
- U8 pad 7: Net-(R59-Pad2) -> Net-(R57-Pad2)
- U9 pad 1: Net-(R61-Pad2) -> Net-(R59-Pad2)
- U9 pad 15: Net-(R60-Pad2) -> Net-(R58-Pad2)
- U9 pad 2: Net-(R62-Pad2) -> Net-(R60-Pad2)
- U9 pad 3: Net-(R63-Pad2) -> Net-(R61-Pad2)
- U9 pad 4: Net-(R64-Pad2) -> Net-(R62-Pad2)
- U9 pad 5: Net-(R65-Pad2) -> Net-(R63-Pad2)
- U9 pad 6: Net-(R66-Pad2) -> Net-(R64-Pad2)
- U9 pad 7: Net-(R67-Pad2) -> Net-(R65-Pad2)
Routing:
- net Net-(R2-Pad2): track 3.81 -> 41.9 mm
- net Net-(R3-Pad2): track 0.00 -> 29.2 mm
- net Net-(R50-Pad2): track 13.8 -> 42.0 mm
- net Net-(R34-Pad2): track 13.8 -> 42.0 mm
- net Net-(R58-Pad2): track 13.8 -> 41.9 mm
- net Net-(R42-Pad2): track 13.8 -> 41.9 mm
- net Net-(R26-Pad2): track 13.8 -> 41.9 mm
- net Net-(R10-Pad2): track 13.8 -> 41.9 mm
- net Net-(R18-Pad2): track 13.8 -> 41.9 mm
- net Net-(D2-Pad2): track 23.0 -> 0.00 mm
- net Net-(R66-Pad1): track 0.00 -> 22.6 mm
- net Net-(R43-Pad2): track 8.89 -> 29.2 mm
- net Net-(R27-Pad2): track 8.89 -> 29.1 mm
- net Net-(R19-Pad2): track 8.89 -> 29.1 mm
- net Net-(R59-Pad2): track 8.89 -> 29.1 mm
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Other:
- board size 180 x 195 mm -> 180 x 200 mm
